File: hardware/Prototyp/Schaltplan_Ultraschallsensor/Schaltplan Ultraschallsensor.kicad_pcb (KiCad board)
At the start: 2 copper layers, 49 parts, among them IC1 A5950, P1 CON-SENSOR2, P2 CONN_01X05, U1 XMC1XXX40, U2 TLC272, U3 LMR62014X, X1 CRYSTAL_3225

Commit message: Layout
Parts:
- removed FILTER1: Filter-4x, kicad-libraries:DFN8-17x135
- removed R14, R15, R16: 56, kicad-libraries:R0603F
- removed R17: 0, kicad-libraries:R0402E
- added C15: 220pF, kicad-libraries:C0402F, F.Cu at (105.6, 69.5)
- added C16: 100nF, kicad-libraries:C0603F, F.Cu at (86.4, 87.9)
- added RP2: 1k, kicad-libraries:0603X4, F.Cu at (108.0, 83.6)
- added RP3: 82, kicad-libraries:4X0402, F.Cu at (106.9, 71.6)
- C13, C14: footprint C0603F -> kicad-libraries:C0603F
- C5, C6, C7, C8: footprint kicad-libraries:C0603F -> kicad-libraries:C0805
- D1: footprint kicad-libraries:SOD-123F -> kicad-libraries:SOD-123
- D2: footprint kicad-libraries:DO-214AA -> kicad-libraries:SOD-123
- L1, L3: footprint kicad-libraries:0603F -> kicad-libraries:C0603F
- L2: footprint kicad-libraries:0603F -> kicad-libraries:NR3030
- U1: value XMC1XXX40 -> XMC1XXX48; footprint kicad-libraries:HVQFN40-6x6 -> kicad-libraries:QFN48-EP2
- moved P1 73.9 mm to (109.8, 63.2), turned to 180 degrees
- moved C10 66.6 mm to (86.0, 94.1), turned to 90 degrees
- moved RP1 65.8 mm to (99.7, 86.1), turned to 180 degrees
- moved R6 63.3 mm to (86.8, 96.3), turned to 180 degrees
- moved R10 63.1 mm to (85.0, 87.9), turned to 90 degrees
- moved P2 62.9 mm to (103.5, 104.0), turned to 0 degrees
- moved R9 62.2 mm to (89.6, 84.4)
- moved R12 62.1 mm to (91.6, 93.3)
- moved C11 61.7 mm to (89.6, 87.2)
- moved R11 60.5 mm to (88.9, 85.8), turned to 0 degrees
- moved R5 59.7 mm to (89.5, 98.9)
- moved D2 59.0 mm to (90.6, 100.5)
- moved LS1 58.7 mm to (118.6, 101.4), turned to 270 degrees
- moved R4 57.6 mm to (92.0, 95.5), turned to 90 degrees
- moved R7 57.0 mm to (86.5, 98.9), turned to 0 degrees
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Connections:
- net +Ua renamed MP+Ua
- net AusA renamed MP-Ausgangsspannung
- net VSspg1 renamed OPV-Zwischenkreis
- C1 pad 1: VCC -> +3V3
- C1 pad 2: GND -> MP-GND
- C10 pad 2: GND -> MP-GND
- C11 pad 2: GND -> MP-GND
- C13 pad 2: GND -> MP-GND
- C14 pad 2: GND -> MP-GND
- C2 pad 1: VCC -> +3V3
- C2 pad 2: GND -> MP-GND
- C3 pad 1: VCC -> +3V3
- C3 pad 2: GND -> MP-GND
- C4 pad 1: VCC -> +3V3
- C4 pad 2: GND -> MP-GND
- C5 pad 1: +3.3VADC -> +5V
- C5 pad 2: GND -> MP-GND
- C6 pad 2: GND -> MP-GND
- C7 pad 2: GND -> MP-GND
- C8 pad 2: GND -> MP-GND
- D2 pad 1: GND -> MP-GND
- IC1 pad 1: GND -> MP-GND
- IC1 pad 11: Net-(IC1-Pad11) -> HB-Phase
- IC1 pad 12: Net-(IC1-Pad12) -> HB-Enable
- IC1 pad 13: Net-(IC1-Pad13) -> HB-Mode
- IC1 pad 2: GND -> MP-GND
- IC1 pad 4: GND -> MP-GND
- IC1 pad 6: GND -> MP-GND
- IC1 pad 8: Net-(IC1-Pad8) -> HB-Reset
- IC1 pad 9: GND -> MP-GND
- L1 pad 1: +3.3VADC -> +5V
- LS1 pad 2: GND -> MP-GND
- P1 pad 2: GND -> MP-GND
- P1 pad 3: +3.3VADC -> +3V3
- P1 pad EP: GND -> MP-GND
- P2 pad 2: VSspg2 -> OPV-Aus
- P2 pad 4: GND -> MP-GND
- R10 pad 1: +5V -> +3V3
- R11 pad 1: VSspg2 -> OPV-Aus
- R11 pad 2: GND -> MP-GND
- R2 pad 2: GND -> MP-GND
- R3 pad 2: /Spannungspumpe/nSHDN -> SP-SHDN
- R4 pad 2: GND -> MP-GND
- R5 pad 2: GND -> MP-GND
- R7 pad 1: +5V -> +3V3
- R9 pad 2: GND -> MP-GND
- RP1 pad 5: GND -> MP-GND
- RP1 pad 6: GND -> MP-GND
- RP1 pad 7: GND -> MP-GND
- RP1 pad 8: GND -> MP-GND
- U1 pad 10: Net-(U1-Pad10) -> Net-(D5-Pad2)
- U1 pad 11: Net-(U1-Pad11) -> Net-(D4-Pad2)
- U1 pad 12: Net-(U1-Pad12) -> Net-(D3-Pad2)
- U1 pad 13: GND -> Net-(U1-Pad13)
- U1 pad 14: VCC -> Net-(U1-Pad14)
- U1 pad 15: VCC -> Net-(U1-Pad15)
- U1 pad 16: S-MISO -> Net-(U1-Pad16)
- U1 pad 17: Net-(U1-Pad17) -> MP-GND
- U1 pad 18: Net-(U1-Pad18) -> +3V3
- U1 pad 19: S-CLK -> +3V3
- U1 pad 20: S-MOSI -> S-MISO
- U1 pad 21: S-CS -> Net-(U1-Pad21)
- U1 pad 23: Net-(IC1-Pad13) -> S-CLK
- U1 pad 24: Net-(IC1-Pad12) -> S-MOSI
- U1 pad 25: Net-(IC1-Pad11) -> S-CS
- U1 pad 26: Net-(IC1-Pad8) -> Net-(U1-Pad26)
- U1 pad 27: VSspg2 -> +3V3
- U1 pad 28: /Spannungspumpe/nSHDN -> Net-(U1-Pad28)
- U1 pad 3: Net-(U1-Pad3) -> SP-SHDN
- U1 pad 31: GND -> Net-(U1-Pad31)
- U1 pad 32: VCC -> Net-(U1-Pad32)
- U1 pad 33: Net-(U1-Pad33) -> OPV-Aus
- U1 pad 35: Net-(C13-Pad1) -> Net-(U1-Pad35)
- U1 pad 37: Net-(U1-Pad37) -> MP-GND
- U1 pad 38: Net-(U1-Pad38) -> +3V3
- U1 pad 4: Net-(D5-Pad2) -> HB-Mode
- U1 pad 5: Net-(D4-Pad2) -> HB-Enable
- U1 pad 6: Net-(D3-Pad2) -> HB-Phase
- U1 pad 7: Net-(U1-Pad7) -> HB-Reset
- U1 pad 8: (no net) -> Net-(U1-Pad8)
- U2 pad 4: GND -> MP-GND
- U2 pad 7: VSspg2 -> OPV-Aus
- U2 pad 8: +5V -> +3V3
- U3 pad 2: GND -> MP-GND
- U3 pad 4: /Spannungspumpe/nSHDN -> SP-SHDN
- X1 pad 3: GND -> MP-GND
Routing:
- net +3V3: track 0.00 -> 110.1 mm, vias 0 -> 4
- net GND: track 73.0 -> 0.00 mm, vias 27 -> 0
- net VSspg2: track 68.1 -> 0.00 mm, vias 4 -> 0
- net MP-GND: track 0.00 -> 49.9 mm, vias 0 -> 41
- net MP-Ausgangsspannung: track 90.2 -> 54.3 mm, vias 3 -> 2
- net MP+Ua: track 70.9 -> 38.3 mm, vias 3 -> 2
- net OPV-Aus: track 0.00 -> 30.8 mm, vias 0 -> 4
- net SP-SHDN: track 0.00 -> 29.9 mm, vias 0 -> 2
- net +3.3VADC: track 28.4 -> 0.00 mm, vias 2 -> 0
- net OPV-Zwischenkreis: track 53.6 -> 26.8 mm
- net +5V: track 29.9 -> 8.94 mm, vias 2 -> 0
- net VCC: track 19.9 -> 0.00 mm, vias 2 -> 0
- net Net-(R12-Pad2): track 26.5 -> 7.13 mm
- net /Spannungspumpe/nSHDN: track 18.0 -> 0.00 mm
- net Net-(C8-Pad1): track 15.1 -> 0.00 mm, vias 2 -> 0
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- added copper zone on B.Cu, net MP-GND
- added copper zone on F.Cu, net MP-GND
- added copper zone on F.Cu, net Net-(C6-Pad1)
- added copper zone on F.Cu, net Net-(C8-Pad1)
- added copper zone on F.Cu, net Net-(D1-Pad2)
- removed copper zone on B.Cu, net GND
Other:
- board outline added: 43.5 x 46.9 mm
- rule pad_to_mask_clearance: 0.2 -> 0

Commit message: platinenlayout
Parts:
- added P3: CONN_01X01, kicad-libraries:DEBUG_PAD, F.Cu at (97.3, 93.7)
- added P4: CONN_01X02, kicad-libraries:SolderJumper, F.Cu at (97.5, 96.0)
- moved C2 12.4 mm to (104.0, 87.9), turned to 0 degrees
- moved C3 5.99 mm to (98.7, 90.7), turned to 90 degrees
Routing:
- net MP-GND: track 49.9 -> 65.3 mm, vias 41 -> 45
- net Net-(P3-Pad1): track 0.00 -> 3.40 mm
- net OPV-Aus: track 30.8 -> 33.5 mm, vias 4 -> 2
- net Net-(P4-Pad1): track 0.00 -> 2.21 mm
- net +3V3: track 110.1 -> 111.9 mm, vias 4 -> 5
Other:
- board text added: "MP+UA"
- board text added: "MP-AUS"
- board text added: "MP-GND"
- board text added: "OPV-Aus"
- board text added: "OPV-Zk"

Commit message: Layout
Parts:
- added R17: 0, kicad-libraries:R0603F, F.Cu at (118.3, 66.1)
- added R18: 0, kicad-libraries:R0603F, F.Cu at (112.0, 79.6)
Connections:
- C5 pad 1: +5V -> Net-(C5-Pad1)
- IC1 pad 5: MP+Ua -> Net-(IC1-Pad5)
- L1 pad 1: +5V -> Net-(C5-Pad1)
Routing:
- net Net-(IC1-Pad5): track 0.00 -> 4.73 mm
- net Net-(C5-Pad1): track 0.00 -> 4.32 mm
- net +5V: track 8.94 -> 4.70 mm
- net MP+Ua: track 38.3 -> 36.4 mm
- net Net-(P4-Pad1): track 2.21 -> 3.90 mm
- net +3V3: track 111.9 -> 113.1 mm

Commit message: Befestigungen
Parts:
- added U5: DRILL, kicad-libraries:DRILL_NP, F.Cu at (90.0, 70.0)
- added U6: DRILL, kicad-libraries:DRILL_NP, F.Cu at (90.0, 105.0)
Changed lines of the file:
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@@
     (tracks 493)
     (zones 0)
-    (modules 52)
+    (modules 54)
     (nets 75)
   )
@@
   (layers
     (0 F.Cu signal)
-    (31 B.Cu signal)
+    (31 B.Cu signal hide)
     (32 B.Adhes user)
     (33 F.Adhes user)
@@
     )
   )
+  (module kicad-libraries:DRILL_NP (layer F.Cu)
+    (at 90 70)
+    (fp_text reference U5 (at 0 0) (layer F.SilkS) hide
+      (effects (font (size 0.29972 0.29972) (thickness 0.0762)))
+    )
+    (fp_text value DRILL (at 0 0.50038) (layer F.SilkS) hide
+      (effects (font (size 0.29972 0.29972) (thickness 0.0762)))
+    )
+    (fp_circle (center 0 0) (end 3.2 0) (layer Eco2.User) (width 0.01))
+    (fp_circle (center 0 0) (end 2.19964 -0.20066) (layer F.SilkS) (width 0.381))
+    (fp_circle (center 0 0) (end 1.99898 -0.20066) (layer F.SilkS) (width 0.381))
+    (fp_circle (center 0 0) (end 1.69926 0) (layer F.SilkS) (width 0.381))
+    (fp_circle (center 0 0) (end 1.39954 -0.09906) (layer B.SilkS) (width 0.381))
+    (fp_circle (center 0 0) (end 1.39954 0) (layer F.SilkS) (width 0.381))
+    (fp_circle (center 0 0) (end 1.69926 0) (layer B.SilkS) (width 0.381))
+    (fp_circle (center 0 0) (end 1.89992 0) (layer B.SilkS) (width 0.381))
+    (fp_circle (center 0 0) (end 2.19964 0) (layer B.SilkS) (width 0.381))
+    (pad "" np_thru_hole circle (at 0 0) (size 2.99974 2.99974) (drill 2.99974) (layers *.Cu *.Mask F.SilkS)
+      (clearance 0.89916))
+  )
+  (module kicad-libraries:DRILL_NP (layer F.Cu)
+    (at 90 105)
+    (fp_text reference U6 (at 0 0) (layer F.SilkS) hide
+      (effects (font (size 0.29972 0.29972) (thickness 0.0762)))
+    )
+    (fp_text value DRILL (at 0 0.50038) (layer F.SilkS) hide
+      (effects (font (size 0.29972 0.29972) (thickness 0.0762)))
+    )
+    (fp_circle (center 0 0) (end 3.2 0) (layer Eco2.User) (width 0.01))
+    (fp_circle (center 0 0) (end 2.19964 -0.20066) (layer F.SilkS) (width 0.381))
+    (fp_circle (center 0 0) (end 1.99898 -0.20066) (layer F.SilkS) (width 0.381))
+    (fp_circle (center 0 0) (end 1.69926 0) (layer F.SilkS) (width 0.381))
+    (fp_circle (center 0 0) (end 1.39954 -0.09906) (layer B.SilkS) (width 0.381))
+    (fp_circle (center 0 0) (end 1.39954 0) (layer F.SilkS) (width 0.381))
+    (fp_circle (center 0 0) (end 1.69926 0) (layer B.SilkS) (width 0.381))
+    (fp_circle (center 0 0) (end 1.89992 0) (layer B.SilkS) (width 0.381))
+    (fp_circle (center 0 0) (end 2.19964 0) (layer B.SilkS) (width 0.381))
+    (pad "" np_thru_hole circle (at 0 0) (size 2.99974 2.99974) (drill 2.99974) (layers *.Cu *.Mask F.SilkS)
+      (clearance 0.89916))
+  )
   (gr_text MP-AUS (at 108.6 107.8 90) (layer F.SilkS)

Commit message: korrekturPCB
Parts:
- moved D4 0.60 mm to (107.6, 87.0)
- moved D3 0.60 mm to (106.2, 87.0)
- moved D5 0.60 mm to (109.0, 87.0)
- moved C13 0.45 mm to (102.6, 100.7)
- moved C14 0.45 mm to (108.0, 100.7)
- moved X1 0.45 mm to (105.3, 100.7)
Connections:
- RP2 pad 1: Net-(RP2-Pad1) -> Net-(D3-Pad1)
- RP2 pad 2: Net-(D3-Pad1) -> Net-(D4-Pad1)
- RP2 pad 3: Net-(D4-Pad1) -> Net-(D5-Pad1)
- RP2 pad 4: Net-(D5-Pad1) -> Net-(RP2-Pad4)
- U1 pad 10: Net-(D5-Pad2) -> Net-(U1-Pad10)
- U1 pad 11: Net-(D4-Pad2) -> Net-(U1-Pad11)
- U1 pad 12: Net-(D3-Pad2) -> Net-(U1-Pad12)
- U1 pad 13: Net-(U1-Pad13) -> Net-(D5-Pad2)
- U1 pad 14: Net-(U1-Pad14) -> Net-(D4-Pad2)
- U1 pad 15: Net-(U1-Pad15) -> Net-(D3-Pad2)
- U1 pad 31: Net-(U1-Pad31) -> OPV-Aus
- U1 pad 33: OPV-Aus -> Net-(U1-Pad33)
- U1 pad 46: Net-(U1-Pad46) -> HB-Enable
- U1 pad 47: Net-(U1-Pad47) -> HB-Phase
- U1 pad 48: Net-(U1-Pad48) -> HB-Reset
- U1 pad 5: HB-Enable -> OPV-Aus
- U1 pad 6: HB-Phase -> Net-(U1-Pad6)
- U1 pad 7: HB-Reset -> Net-(U1-Pad7)
Routing:
- net OPV-Aus: track 33.5 -> 42.6 mm
- net HB-Enable: track 8.17 -> 14.5 mm
- net HB-Reset: track 11.2 -> 17.5 mm
- net HB-Phase: track 7.25 -> 12.9 mm
- net Net-(D5-Pad2): track 5.32 -> 3.38 mm
- net Net-(D4-Pad2): track 4.23 -> 3.03 mm
- net Net-(D3-Pad2): track 3.20 -> 2.01 mm
- net MP+Ua: track 36.4 -> 37.4 mm
- net MP-GND: track 65.7 -> 65.0 mm
- net HB-Mode: track 9.06 -> 9.36 mm, vias 0 -> 2
- net SP-SHDN: vias 2 -> 4
