File: hardware/Prototyp/Schaltplan_Ultraschallsensor/Schaltplan Ultraschallsensor.sch (KiCad schematic (older format))
At the start: 9 parts, among them IC1 A5950, J1 Conn_01x06_Female, P1 CON-SENSOR2, U1 XMC1XXX40

Commit message: Schaltplanaktualisierung
Parts:
- removed J1: Conn_01x06_Female, symbol Conn_01x06_Female
- added C13, C14: 10pF, C0603F, symbol C
- added D3, D5: Gelb, kicad-libraries:D0603E, symbol LED
- added D4: Gleb, kicad-libraries:D0603E, symbol LED
- added FILTER1: Filter-4x, kicad-libraries:DFN8-17x135, symbol Filter-4x
- added P2: CONN_01X05, kicad-libraries:pin_array_5x1, symbol CONN_01X05
- added R14, R15, R16: 56, kicad-libraries:R0603F, symbol R
- added R17: 0, kicad-libraries:R0402E, symbol R
- added RP1: 10k, kicad-libraries:0603X4, symbol R_PACK4
- added X1: CRYSTAL_3225, kicad-libraries:CRYSTAL_3225, symbol CRYSTAL_3225
- C1, C2, C3, C4: footprint C0603F -> kicad-libraries:C0603F
- IC1: footprint (none) -> Zusatzteile:16-leadTSSOP_0,137,4,4mmBreite
- LS1: footprint (none) -> Zusatzteile:Ultraschallsensor
- P1: footprint CON-SENSOR2 -> kicad-libraries:CON-SENSOR2
- U1: footprint (none) -> kicad-libraries:HVQFN40-6x6
Connections:
- net labels added: +3.3VADC, S-CLK, S-CS, S-MISO, S-MOSI
- net labels removed: +3V3, AusB
- wire segments 82 -> 132
- no-connect marks 39 -> 27
Other:
- moved on the sheet: P1, U1B, U1C

Commit message: Platinenlayout
Connections:
- net at U1.29 (P0.6): no longer D5.2 (K)
- net at U1.30 (P0.7), U1.?? (VSSP): no longer D4.2 (K)
- net at U1.33 (P0.8): no longer D3.2 (K)
- net at U1.4 (P2.3): now also D5.2 (K)
- net at U1.5 (P2.4): now also D4.2 (K)
- net at U1.6 (P2.5): now also D3.2 (K)
- no-connect marks 27 -> 26
Other:
- moved on the sheet: D3, D4, D5, R14, R15, R16, U1D
Changed lines of the file:
@@
 L XMC1XXX40 U1
 U 4 1 5A70A99D
-P 6600 6950
-F 0 "U1" H 6400 7650 60  0000 C CNN
-F 1 "XMC1XXX40" H 6600 6250 60  0000 C CNN
-F 2 "kicad-libraries:HVQFN40-6x6" H 6750 7700 60  0001 C CNN
-F 3 "" H 6750 7700 60  0000 C CNN
-	4    6600 6950
+P 10300 2750
+F 0 "U1" H 10100 3450 60  0000 C CNN
+F 1 "XMC1XXX40" H 10300 2050 60  0000 C CNN
+F 2 "kicad-libraries:HVQFN40-6x6" H 10450 3500 60  0001 C CNN
+F 3 "" H 10450 3500 60  0000 C CNN
+	4    10300 2750
 	1    0    0    -1
 $EndComp
@@
 	3450 1850 3450 3450
 Connection ~ 7150 1900
-NoConn ~ 6250 7450
-NoConn ~ 6250 7350
-NoConn ~ 6250 7250
-NoConn ~ 6250 7150
-NoConn ~ 6250 7050
-NoConn ~ 6250 6950
-NoConn ~ 6250 6900
-NoConn ~ 6250 6850
-NoConn ~ 6250 6750
-NoConn ~ 6250 6650
-NoConn ~ 6250 6550
-NoConn ~ 6250 6450
+NoConn ~ 9950 3250
+NoConn ~ 9950 3150
+NoConn ~ 9950 3050
+NoConn ~ 9950 2950
+NoConn ~ 9950 2850
+NoConn ~ 9950 2700
+NoConn ~ 9950 2450
+NoConn ~ 9950 2350
+NoConn ~ 9950 2250
 NoConn ~ 5400 7000
 NoConn ~ 5400 6900
@@
 L LED D5
 U 1 1 5A7323BC
-P 3600 3900
-F 0 "D5" H 3600 4000 50  0000 C CNN
-F 1 "Gelb" H 3750 4000 50  0000 C CNN
-F 2 "kicad-libraries:D0603E" H 3600 3900 50  0001 C CNN
-F 3 "" H 3600 3900 50  0000 C CNN
-	1    3600 3900
+P 8900 2450
+F 0 "D5" H 8900 2550 50  0000 C CNN
+F 1 "Gelb" H 9050 2550 50  0000 C CNN
+F 2 "kicad-libraries:D0603E" H 8900 2450 50  0001 C CNN
+F 3 "" H 8900 2450 50  0000 C CNN
+	1    8900 2450
 	1    0    0    -1
 $EndComp
@@
 L LED D4
 U 1 1 5A732455
-P 3600 4100
-F 0 "D4" H 3600 4200 50  0000 C CNN
-F 1 "Gleb" H 3750 4200 50  0000 C CNN
-F 2 "kicad-libraries:D0603E" H 3600 4100 50  0001 C CNN
-F 3 "" H 3600 4100 50  0000 C CNN
-	1    3600 4100
+P 8900 2650
+F 0 "D4" H 8900 2750 50  0000 C CNN
+F 1 "Gleb" H 9050 2750 50  0000 C CNN
+F 2 "kicad-libraries:D0603E" H 8900 2650 50  0001 C CNN
+F 3 "" H 8900 2650 50  0000 C CNN
+	1    8900 2650
 	1    0    0    -1
 $EndComp
@@
 L LED D3
 U 1 1 5A7324B4
-P 3600 4300
-F 0 "D3" H 3600 4400 50  0000 C CNN
-F 1 "Gelb" H 3750 4400 50  0000 C CNN
-F 2 "kicad-libraries:D0603E" H 3600 4300 50  0001 C CNN
-F 3 "" H 3600 4300 50  0000 C CNN
-	1    3600 4300
-	1    0    0    -1
-$EndComp
-Wire Wire Line
-	2750 3800 2750 4300
-Wire Wire Line
-	2750 4100 2800 4100
-Connection ~ 2750 3900
-Wire Wire Line
-	2750 4300 2800 4300
-Connection ~ 2750 4100
-Wire Wire Line
-	2800 3900 2750 3900
+P 8900 2850
+F 0 "D3" H 8900 2950 50  0000 C CNN
+F 1 "Gelb" H 9050 2950 50  0000 C CNN
+F 2 "kicad-libraries:D0603E" H 8900 2850 50  0001 C CNN
+F 3 "" H 8900 2850 50  0000 C CNN
+	1    8900 2850
+	1    0    0    -1
+$EndComp
+Wire Wire Line
+	8050 2350 8050 2850
+Wire Wire Line
+	8050 2650 8100 2650
+Connection ~ 8050 2450
+Wire Wire Line
+	8050 2850 8100 2850
+Connection ~ 8050 2650
+Wire Wire Line
+	8100 2450 8050 2450
 $Comp
 L R R14
 U 1 1 5A74243E
-P 3050 3900
-F 0 "R14" V 3130 3900 50  0000 C CNN
-F 1 "56" V 3050 3900 50  0000 C CNN
-F 2 "kicad-libraries:R0603F" H 3050 3900 60  0001 C CNN
-F 3 "" H 3050 3900 60  0000 C CNN
-	1    3050 3900
+P 8350 2450
+F 0 "R14" V 8430 2450 50  0000 C CNN
+F 1 "56" V 8350 2450 50  0000 C CNN
+F 2 "kicad-libraries:R0603F" H 8350 2450 60  0001 C CNN
+F 3 "" H 8350 2450 60  0000 C CNN
+	1    8350 2450
 	0    1    1    0
 $EndComp
@@
 L R R15
 U 1 1 5A742BF8
-P 3050 4100
-F 0 "R15" V 3130 4100 50  0000 C CNN
-F 1 "56" V 3050 4100 50  0000 C CNN
-F 2 "kicad-libraries:R0603F" H 3050 4100 60  0001 C CNN
-F 3 "" H 3050 4100 60  0000 C CNN
-	1    3050 4100
+P 8350 2650
+F 0 "R15" V 8430 2650 50  0000 C CNN
+F 1 "56" V 8350 2650 50  0000 C CNN
+F 2 "kicad-libraries:R0603F" H 8350 2650 60  0001 C CNN
+F 3 "" H 8350 2650 60  0000 C CNN
+	1    8350 2650
 	0    1    1    0
 $EndComp
@@
 L R R16
 U 1 1 5A742C8A
-P 3050 4300
-F 0 "R16" V 3130 4300 50  0000 C CNN
-F 1 "56" V 3050 4300 50  0000 C CNN
-F 2 "kicad-libraries:R0603F" H 3050 4300 60  0001 C CNN
-F 3 "" H 3050 4300 60  0000 C CNN
-	1    3050 4300
+P 8350 2850
+F 0 "R16" V 8430 2850 50  0000 C CNN
+F 1 "56" V 8350 2850 50  0000 C CNN
+F 2 "kicad-libraries:R0603F" H 8350 2850 60  0001 C CNN
+F 3 "" H 8350 2850 60  0000 C CNN
+	1    8350 2850
 	0    1    1    0
 $EndComp
 Wire Wire Line
-	3300 3900 3400 3900
-Wire Wire Line
-	3400 4100 3300 4100
-Wire Wire Line
-	3300 4300 3400 4300
+	8600 2450 8700 2450
+Wire Wire Line
+	8700 2650 8600 2650
+Wire Wire Line
+	8600 2850 8700 2850
 $Comp
 L +3.3VADC #PWR019
@@
 L +3.3VADC #PWR021
 U 1 1 5A744D41
-P 2750 3800
-F 0 "#PWR021" H 2900 3750 50  0001 C CNN
-F 1 "+3.3VADC" H 2750 3900 50  0000 C CNN
-F 2 "" H 2750 3800 50  0001 C CNN
-F 3 "" H 2750 3800 50  0001 C CNN
-	1    2750 3800
+P 8050 2350
+F 0 "#PWR021" H 8200 2300 50  0001 C CNN
+F 1 "+3.3VADC" H 8050 2450 50  0000 C CNN
+F 2 "" H 8050 2350 50  0001 C CNN
+F 3 "" H 8050 2350 50  0001 C CNN
+	1    8050 2350
 	1    0    0    -1
 $EndComp
@@
 	5300 4250 5600 4250
 Wire Wire Line
-	3800 3900 3850 3900
-Wire Wire Line
-	3850 3900 3850 3850
-Wire Wire Line
-	3850 3850 5600 3850
-Wire Wire Line
-	3800 4100 3900 4100
-Wire Wire Line
-	3900 4100 3900 3950
-Wire Wire Line
-	3900 3950 5600 3950
-Wire Wire Line
-	3800 4300 3950 4300
-Wire Wire Line
-	3950 4300 3950 4050
-Wire Wire Line
-	3950 4050 5600 4050
+	9100 2450 9150 2450
+Wire Wire Line
+	9100 2650 9950 2650
 NoConn ~ 5600 4150
 NoConn ~ 5600 4450
@@
 	5050 7100 5400 7100
 NoConn ~ 5050 7200
+NoConn ~ 5600 3850
+NoConn ~ 5600 4050
+Wire Wire Line
+	9950 2550 9150 2550
+Wire Wire Line
+	9150 2550 9150 2450
+Wire Wire Line
+	9100 2850 9150 2850
+Wire Wire Line
+	9150 2850 9150 2750
+Wire Wire Line
+	9150 2750 9950 2750
 $EndSCHEMATC

Commit message: Layout
Parts:
- removed FILTER1: Filter-4x, kicad-libraries:DFN8-17x135, symbol Filter-4x
- removed R14, R15, R16: 56, kicad-libraries:R0603F, symbol R
- removed R17: 0, kicad-libraries:R0402E, symbol R
- removed U1: XMC1XXX40, kicad-libraries:HVQFN40-6x6, symbol XMC1XXX40
- added C15: 220pF, kicad-libraries:C0402F, symbol C
- added RP2: 1k, kicad-libraries:0603X4, symbol R_PACK4
- added RP3: 82, kicad-libraries:4X0402, symbol R_PACK4
- added U1: XMC1XXX48, kicad-libraries:QFN48-EP2, symbol XMC1XXX48
- C13, C14: footprint C0603F -> kicad-libraries:C0603F
Connections:
- net VCC is gone; now on net +3V3: C1.1, C2.1, C3.1, C4.1
- net GND: now also C15.2, U1.17 (VSS), U1.37 (VSSP), U1.EP (VSSP)
- net S-CLK: now also RP3.3 (P3), U1.23 (P1.3_IHO)
- net S-CS: now also RP3.4 (P4), U1.25 (P1.1_IHO)
- net S-MISO: now also RP3.1 (P1), U1.20 (P1.6_IHO)
- net S-MOSI: now also RP3.2 (P2), U1.24 (P1.2_IHO)
- net HB-Mode: now reaches IC1.13 (Mode)
- net HB-Mode: now also U1.4 (P2.1_AIO)
- net HB-Enable: now reaches IC1.12 (Enable)
- net HB-Enable: now also U1.5 (P2.2_AI)
- net HB-Phase: now reaches IC1.11 (Phase)
- net HB-Phase: now also U1.6 (P2.3_AI)
- net HB-Reset: now reaches IC1.8 (RESTn)
- net HB-Reset: now also U1.7 (P2.4_AI)
- net at C13.1, X1.2: now also U1.41 (P0.10_IO/XTAL1)
- net at D5.2 (K): now also U1.10 (P2.7_AI)
- net at D4.2 (K): now also U1.11 (P2.8_AI)
- net at D3.2 (K): now also U1.12 (P2.9_AI)
- net at P1.4 (CS): now also RP3.5 (R4)
- net at P1.5 (CLK): now also RP3.6 (R3)
- net at P1.6 (MOSI): now also RP3.7 (R2)
- net at P1.7 (MISO): now also C15.1, RP3.8 (R1)
- net at D5.1 (A): now also RP2.4 (P4)
- net at D4.1 (A): now also RP2.3 (P3)
- net at D3.1 (A): now also RP2.2 (P2)
- net at C14.1, X1.1: now also U1.42 (P0.11_IO/XTAL2)
- net +3.3VADC renamed +3V3
- net +3V3: now also RP2.5 (R4), RP2.6 (R3), RP2.7 (R2), RP2.8 (R1), U1.18 (VDD), U1.19 (VDDP), U1.27 (VDDP), U1.38 (VDDP)
- net +Ua renamed MP+Ua
- net AusA renamed MP-Ausgangsspannung
- net VSspg1 renamed OPV-Zwischenkreis
- net VSspg2 renamed OPV-Aus
- net OPV-Aus: now also U1.33 (P0.4_IO)
- new net SP-SHDN: U1.3 (P2.0_AIO)
- no-connect marks 26 -> 34
Other:
- moved on the sheet: C13, C14, P2, X1

Commit message: platinenlayout
Parts:
- added P3: CONN_01X01, kicad-libraries:DEBUG_PAD, symbol CONN_01X01
- added P4: CONN_01X02, kicad-libraries:SolderJumper, symbol CONN_01X02
Connections:
- net GND: now also P4.2 (P2)
- net at U1.34 (P0.5_IO): now also P3.1 (P1)
- net at U1.36 (P0.7_IO): now also P4.1 (P1)
- no-connect marks 34 -> 32
Changed lines of the file:
@@
 	1    0    0    -1
 $EndComp
-NoConn ~ 5600 3950
 NoConn ~ 9950 3050
 NoConn ~ 9950 2950
@@
 Wire Wire Line
 	9950 2250 9800 2250
-NoConn ~ 5600 3750
+$Comp
+L CONN_01X02 P4
+U 1 1 5A79D172
+P 5150 4000
+F 0 "P4" H 5350 4000 50  0000 C CNN
+F 1 "CONN_01X02" H 5500 4100 50  0000 C CNN
+F 2 "kicad-libraries:SolderJumper" H 5150 4000 50  0001 C CNN
+F 3 "" H 5150 4000 50  0000 C CNN
+	1    5150 4000
+	-1   0    0    -1
+$EndComp
+$Comp
+L CONN_01X01 P3
+U 1 1 5A79D279
+P 5150 3750
+F 0 "P3" H 5350 3700 50  0000 C CNN
+F 1 "CONN_01X01" H 5500 3800 50  0000 C CNN
+F 2 "kicad-libraries:DEBUG_PAD" H 5150 3750 50  0001 C CNN
+F 3 "" H 5150 3750 50  0000 C CNN
+	1    5150 3750
+	-1   0    0    1
+$EndComp
+Wire Wire Line
+	5350 3750 5600 3750
+Wire Wire Line
+	5350 3950 5600 3950
+$Comp
+L GND #PWR020
+U 1 1 5A79E6E5
+P 5400 4100
+F 0 "#PWR020" H 5400 4100 30  0001 C CNN
+F 1 "GND" H 5400 4030 30  0001 C CNN
+F 2 "" H 5400 4100 60  0000 C CNN
+F 3 "" H 5400 4100 60  0000 C CNN
+	1    5400 4100
+	1    0    0    -1
+$EndComp
+Wire Wire Line
+	5350 4050 5400 4050
+Wire Wire Line
+	5400 4050 5400 4100
 $EndSCHEMATC

Commit message: Layout
Parts:
- added R18: 0, kicad-libraries:R0603F, symbol R
Connections:
- net MP+Ua: now also R18.1; no longer IC1.5 (VBB)
- new net: IC1.5 (VBB), R18.2
Changed lines of the file:
@@
 Connection ~ 7150 1900
 Wire Wire Line
-	5250 1300 5150 1300
-Wire Wire Line
-	5250 900  5250 1300
-Wire Wire Line
-	2650 900  5250 900
+	2650 900  5750 900
 Wire Wire Line
 	2650 900  2650 3300
@@
 Wire Wire Line
 	5400 4050 5400 4100
+$Comp
+L R R18
+U 1 1 5A795B29
+P 5450 1300
+F 0 "R18" V 5530 1300 50  0000 C CNN
+F 1 "0" V 5450 1300 50  0000 C CNN
+F 2 "kicad-libraries:R0603F" H 5450 1300 60  0000 C CNN
+F 3 "" H 5450 1300 60  0000 C CNN
+	1    5450 1300
+	0    1    1    0
+$EndComp
+Wire Wire Line
+	5150 1300 5200 1300
+Wire Wire Line
+	5750 900  5750 1300
+Wire Wire Line
+	5750 1300 5700 1300
 $EndSCHEMATC

Commit message: korrekturPCB
Connections:
- net HB-Enable: now also U1.46 (P0.15_IO); no longer U1.5 (P2.2_AI)
- net HB-Phase: now also U1.47 (P4.4_IO); no longer U1.6 (P2.3_AI)
- net HB-Reset: now also U1.48 (P4.5_IO); no longer U1.7 (P2.4_AI)
- net OPV-Aus: now also U1.31 (P0.2_IO), U1.5 (P2.2_AI); no longer U1.33 (P0.4_IO)
- net at D5.1 (A): now also RP2.3 (P3); no longer RP2.4 (P4)
- net at D5.2 (K): now also U1.13 (P2.10/AIO); no longer U1.10 (P2.7_AI)
- net at D4.1 (A): now also RP2.2 (P2); no longer RP2.3 (P3)
- net at D4.2 (K): now also U1.14 (P2.11/AIO); no longer U1.11 (P2.8_AI)
- net at D3.1 (A): now also RP2.1 (P1); no longer RP2.2 (P2)
- net at D3.2 (K): now also U1.15 (P2.12/AIO); no longer U1.12 (P2.9_AI)
- no-connect marks 32 -> 31
Other:
- moved on the sheet: D3, D4, D5, RP1, RP2, U1C, U1E
