File: hardware/Prototyp/Schaltplan_Ultraschallsensor/Testzeichnung.sch (KiCad schematic (older format))
At the start: 13 parts, among them U3 LMR62014X

Commit message: Schaltplanaktualisierung
Parts:
- added R13: 20k, kicad-libraries:R0603F, symbol R
- C5, C6, C7, C8, C9: footprint C0603F -> kicad-libraries:C0603F
- D1: footprint (none) -> kicad-libraries:SOD-123F
- L1, L2, L3: footprint (none) -> kicad-libraries:0603F
- R1: footprint (none) -> Zusatzteile:ST4ETA
- R2, R3: footprint R0603F -> kicad-libraries:R0603F
- U3: footprint (none) -> kicad-libraries:SOT23-5
Connections:
- net at C8.1, C9.2, D1.1 (K)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: now also R13.1; no longer R1.1
- net +3V3 renamed +3.3VADC
- new net: R1.1, R13.2
Other:
- moved on the sheet: R1
Changed lines of the file:
@@
 F 0 "L1" H 5100 1350 50  0000 C CNN
 F 1 "FB" H 5100 1500 50  0000 C CNN
-F 2 "" H 5250 1400 50  0000 C CNN
+F 2 "kicad-libraries:0603F" H 5250 1400 50  0001 C CNN
 F 3 "" H 5250 1400 50  0000 C CNN
 	1    5250 1400
@@
 F 0 "L2" H 6500 1350 50  0000 C CNN
 F 1 "10uH" H 6550 1500 50  0000 C CNN
-F 2 "" H 6650 1400 50  0000 C CNN
+F 2 "kicad-libraries:0603F" H 6650 1400 50  0001 C CNN
 F 3 "" H 6650 1400 50  0000 C CNN
 	1    6650 1400
@@
 F 0 "L3" H 8650 1350 50  0000 C CNN
 F 1 "FB" H 8650 1500 50  0000 C CNN
-F 2 "" H 8800 1400 50  0000 C CNN
+F 2 "kicad-libraries:0603F" H 8800 1400 50  0001 C CNN
 F 3 "" H 8800 1400 50  0000 C CNN
 	1    8800 1400
@@
 F 0 "C5" H 4825 2000 50  0000 L CNN
 F 1 "4.7uF" H 4825 1800 50  0000 L CNN
-F 2 "C0603F" H 4838 1750 50  0000 C CNN
+F 2 "kicad-libraries:C0603F" H 4838 1750 50  0001 C CNN
 F 3 "" H 4800 1900 50  0000 C CNN
 	1    4800 1900
@@
 F 0 "C6" H 5825 2050 50  0000 L CNN
 F 1 "4.7uF" H 5825 1850 50  0000 L CNN
-F 2 "C0603F" H 5838 1800 50  0000 C CNN
+F 2 "kicad-libraries:C0603F" H 5838 1800 50  0001 C CNN
 F 3 "" H 5800 1950 50  0000 C CNN
 	1    5800 1950
@@
 F 0 "R3" V 6180 1750 50  0000 C CNN
 F 1 "1M" V 6100 1750 50  0000 C CNN
-F 2 "R0603F" V 6030 1750 50  0000 C CNN
+F 2 "kicad-libraries:R0603F" V 6030 1750 50  0001 C CNN
 F 3 "" H 6100 1750 50  0000 C CNN
 	1    6100 1750
@@
 F 0 "D1" H 7550 1500 50  0000 C CNN
 F 1 "B0520LW" H 7550 1300 50  0000 C CNN
-F 2 "" H 7550 1400 50  0000 C CNN
+F 2 "kicad-libraries:SOD-123F" H 7550 1400 50  0001 C CNN
 F 3 "" H 7550 1400 50  0000 C CNN
 	1    7550 1400
@@
 F 0 "R2" V 7380 2400 50  0000 C CNN
 F 1 "13.3k" V 7300 2400 50  0000 C CNN
-F 2 "R0603F" V 7230 2400 50  0000 C CNN
+F 2 "kicad-libraries:R0603F" V 7230 2400 50  0001 C CNN
 F 3 "" H 7300 2400 50  0000 C CNN
 	1    7300 2400
@@
 F 0 "C9" V 8000 2100 50  0000 L CNN
 F 1 "270pF" V 8000 1700 50  0000 L CNN
-F 2 "C0603F" H 7988 1850 50  0000 C CNN
+F 2 "kicad-libraries:C0603F" H 8200 1900 50  0001 C CNN
 F 3 "" H 7950 2000 50  0000 C CNN
 	1    7950 2000
@@
 F 0 "C8" H 8525 2050 50  0000 L CNN
 F 1 "4.7uF" H 8525 1850 50  0000 L CNN
-F 2 "C0603F" H 8538 1800 50  0000 C CNN
+F 2 "kicad-libraries:C0603F" H 8538 1800 50  0001 C CNN
 F 3 "" H 8500 1950 50  0000 C CNN
 	1    8500 1950
@@
 F 0 "C7" H 9125 2050 50  0000 L CNN
 F 1 "4.7uF" H 9125 1850 50  0000 L CNN
-F 2 "C0603F" H 9138 1800 50  0000 C CNN
+F 2 "kicad-libraries:C0603F" H 9138 1800 50  0001 C CNN
 F 3 "" H 9100 1950 50  0000 C CNN
 	1    9100 1950
@@
 $EndComp
 $Comp
-L GND #PWR025
+L GND #PWR031
 U 1 1 5A4CF13E
 P 4800 2700
-F 0 "#PWR025" H 4800 2450 50  0001 C CNN
+F 0 "#PWR031" H 4800 2450 50  0001 C CNN
 F 1 "GND" H 4800 2550 50  0000 C CNN
 F 2 "" H 4800 2700 50  0000 C CNN
@@
 $EndComp
 $Comp
-L GND #PWR026
+L GND #PWR032
 U 1 1 5A4CF1BC
 P 5800 2700
-F 0 "#PWR026" H 5800 2450 50  0001 C CNN
+F 0 "#PWR032" H 5800 2450 50  0001 C CNN
 F 1 "GND" H 5800 2550 50  0000 C CNN
 F 2 "" H 5800 2700 50  0000 C CNN
@@
 $EndComp
 $Comp
-L GND #PWR027
+L GND #PWR033
 U 1 1 5A4CF1EB
 P 6650 2700
-F 0 "#PWR027" H 6650 2450 50  0001 C CNN
+F 0 "#PWR033" H 6650 2450 50  0001 C CNN
 F 1 "GND" H 6650 2550 50  0000 C CNN
 F 2 "" H 6650 2700 50  0000 C CNN
@@
 $EndComp
 $Comp
-L GND #PWR028
+L GND #PWR034
 U 1 1 5A4CF21A
 P 7300 2700
-F 0 "#PWR028" H 7300 2450 50  0001 C CNN
+F 0 "#PWR034" H 7300 2450 50  0001 C CNN
 F 1 "GND" H 7300 2550 50  0000 C CNN
 F 2 "" H 7300 2700 50  0000 C CNN
@@
 $EndComp
 $Comp
-L GND #PWR029
+L GND #PWR035
 U 1 1 5A4CF249
 P 8500 2700
-F 0 "#PWR029" H 8500 2450 50  0001 C CNN
+F 0 "#PWR035" H 8500 2450 50  0001 C CNN
 F 1 "GND" H 8500 2550 50  0000 C CNN
 F 2 "" H 8500 2700 50  0000 C CNN
@@
 $EndComp
 $Comp
-L GND #PWR030
+L GND #PWR036
 U 1 1 5A4CF278
 P 9100 2700
-F 0 "#PWR030" H 9100 2450 50  0001 C CNN
+F 0 "#PWR036" H 9100 2450 50  0001 C CNN
 F 1 "GND" H 9100 2550 50  0000 C CNN
 F 2 "" H 9100 2700 50  0000 C CNN
@@
 F 0 "U3" H 6350 1700 60  0000 C CNN
 F 1 "LMR62014X" H 6950 1700 60  0000 C CNN
-F 2 "" H 6650 2000 60  0000 C CNN
+F 2 "kicad-libraries:SOT23-5" H 6650 2000 60  0001 C CNN
 F 3 "" H 6650 2000 60  0000 C CNN
 	1    6650 2000
@@
 	9100 1750 9100 1400
 $Comp
-L +3V3 #PWR031
-U 1 1 5A6ED2AD
-P 4800 1250
-F 0 "#PWR031" H 4800 1100 50  0001 C CNN
-F 1 "+3V3" H 4800 1390 50  0000 C CNN
-F 2 "" H 4800 1250 50  0001 C CNN
-F 3 "" H 4800 1250 50  0001 C CNN
-	1    4800 1250
-	1    0    0    -1
-$EndComp
-$Comp
 L R_Variable R1
 U 1 1 5A6ED69F
-P 7650 1700
-F 0 "R1" V 7800 1650 50  0000 L CNN
-F 1 "0-200K" V 7550 1650 50  0000 L CNN
-F 2 "" V 7580 1700 50  0001 C CNN
-F 3 "" H 7650 1700 50  0001 C CNN
-	1    7650 1700
+P 7500 1700
+F 0 "R1" V 7650 1650 50  0000 L CNN
+F 1 "0-200K" V 7400 1650 50  0000 L CNN
+F 2 "Zusatzteile:ST4ETA" V 7430 1700 50  0001 C CNN
+F 3 "" H 7500 1700 50  0001 C CNN
+	1    7500 1700
 	0    1    1    0
 $EndComp
@@
 Wire Wire Line
 	6100 2000 6100 2200
-Wire Wire Line
-	7800 1700 8250 1700
-Wire Wire Line
-	7500 1700 7300 1700
+$Comp
+L R R13
+U 1 1 5A72FBF8
+P 7950 1700
+F 0 "R13" V 8030 1700 50  0000 C CNN
+F 1 "20k" V 7950 1700 50  0000 C CNN
+F 2 "kicad-libraries:R0603F" H 7950 1700 60  0001 C CNN
+F 3 "" H 7950 1700 60  0000 C CNN
+	1    7950 1700
+	0    1    1    0
+$EndComp
+Wire Wire Line
+	8200 1700 8250 1700
+Wire Wire Line
+	7650 1700 7700 1700
+Wire Wire Line
+	7300 1700 7350 1700
+$Comp
+L +3.3VADC #PWR037
+U 1 1 5A7450C0
+P 4800 1250
+F 0 "#PWR037" H 4950 1200 50  0001 C CNN
+F 1 "+3.3VADC" H 4800 1350 50  0000 C CNN
+F 2 "" H 4800 1250 50  0001 C CNN
+F 3 "" H 4800 1250 50  0001 C CNN
+	1    4800 1250
+	1    0    0    -1
+$EndComp
 $EndSCHEMATC

Commit message: Platinenlayout
Parts:
- removed R1: 0-200K, Zusatzteile:ST4ETA, symbol R_Variable
- added RV1: 200k, Zusatzteile:ST4ETA, symbol POT
Connections:
- net at C9.1, R2.1, U3.3 (FB): now also RV1.2, RV1.3
- net at R13.2: now also RV1.1
Changed lines of the file:
@@
 Wire Wire Line
 	9100 1750 9100 1400
-$Comp
-L R_Variable R1
-U 1 1 5A6ED69F
-P 7500 1700
-F 0 "R1" V 7650 1650 50  0000 L CNN
-F 1 "0-200K" V 7400 1650 50  0000 L CNN
-F 2 "Zusatzteile:ST4ETA" V 7430 1700 50  0001 C CNN
-F 3 "" H 7500 1700 50  0001 C CNN
-	1    7500 1700
-	0    1    1    0
-$EndComp
 Wire Wire Line
 	6650 2350 6650 2700
@@
 	1    0    0    -1
 $EndComp
+$Comp
+L POT RV1
+U 1 1 5A746D57
+P 7500 1700
+F 0 "RV1" V 7325 1700 50  0000 C CNN
+F 1 "200k" V 7400 1700 50  0000 C CNN
+F 2 "Zusatzteile:ST4ETA" H 7500 1700 50  0001 C CNN
+F 3 "" H 7500 1700 50  0001 C CNN
+	1    7500 1700
+	0    1    1    0
+$EndComp
+Wire Wire Line
+	7500 1850 7300 1850
+Connection ~ 7300 1850
 $EndSCHEMATC

Commit message: Layout
Parts:
- C5, C6, C7, C8: footprint kicad-libraries:C0603F -> kicad-libraries:C0805
- D1: footprint kicad-libraries:SOD-123F -> kicad-libraries:SOD-123
- L1, L3: footprint kicad-libraries:0603F -> kicad-libraries:C0603F
- L2: footprint kicad-libraries:0603F -> kicad-libraries:NR3030
Connections:
- net +3.3VADC renamed +5V
Changed lines of the file:
@@
 F 0 "L1" H 5100 1350 50  0000 C CNN
 F 1 "FB" H 5100 1500 50  0000 C CNN
-F 2 "kicad-libraries:0603F" H 5250 1400 50  0001 C CNN
+F 2 "kicad-libraries:C0603F" H 5250 1400 50  0001 C CNN
 F 3 "" H 5250 1400 50  0000 C CNN
 	1    5250 1400
@@
 F 0 "L2" H 6500 1350 50  0000 C CNN
 F 1 "10uH" H 6550 1500 50  0000 C CNN
-F 2 "kicad-libraries:0603F" H 6650 1400 50  0001 C CNN
+F 2 "kicad-libraries:NR3030" H 6650 1400 50  0001 C CNN
 F 3 "" H 6650 1400 50  0000 C CNN
 	1    6650 1400
@@
 F 0 "L3" H 8650 1350 50  0000 C CNN
 F 1 "FB" H 8650 1500 50  0000 C CNN
-F 2 "kicad-libraries:0603F" H 8800 1400 50  0001 C CNN
+F 2 "kicad-libraries:C0603F" H 8800 1400 50  0001 C CNN
 F 3 "" H 8800 1400 50  0000 C CNN
 	1    8800 1400
@@
 F 0 "C5" H 4825 2000 50  0000 L CNN
 F 1 "4.7uF" H 4825 1800 50  0000 L CNN
-F 2 "kicad-libraries:C0603F" H 4838 1750 50  0001 C CNN
+F 2 "kicad-libraries:C0805" H 4838 1750 50  0001 C CNN
 F 3 "" H 4800 1900 50  0000 C CNN
 	1    4800 1900
@@
 F 0 "C6" H 5825 2050 50  0000 L CNN
 F 1 "4.7uF" H 5825 1850 50  0000 L CNN
-F 2 "kicad-libraries:C0603F" H 5838 1800 50  0001 C CNN
+F 2 "kicad-libraries:C0805" H 5838 1800 50  0001 C CNN
 F 3 "" H 5800 1950 50  0000 C CNN
 	1    5800 1950
@@
 F 0 "D1" H 7550 1500 50  0000 C CNN
 F 1 "B0520LW" H 7550 1300 50  0000 C CNN
-F 2 "kicad-libraries:SOD-123F" H 7550 1400 50  0001 C CNN
+F 2 "kicad-libraries:SOD-123" H 7550 1400 50  0001 C CNN
 F 3 "" H 7550 1400 50  0000 C CNN
 	1    7550 1400
@@
 F 0 "C8" H 8525 2050 50  0000 L CNN
 F 1 "4.7uF" H 8525 1850 50  0000 L CNN
-F 2 "kicad-libraries:C0603F" H 8538 1800 50  0001 C CNN
+F 2 "kicad-libraries:C0805" H 8538 1800 50  0001 C CNN
 F 3 "" H 8500 1950 50  0000 C CNN
 	1    8500 1950
@@
 F 0 "C7" H 9125 2050 50  0000 L CNN
 F 1 "4.7uF" H 9125 1850 50  0000 L CNN
-F 2 "kicad-libraries:C0603F" H 9138 1800 50  0001 C CNN
+F 2 "kicad-libraries:C0805" H 9138 1800 50  0001 C CNN
 F 3 "" H 9100 1950 50  0000 C CNN
 	1    9100 1950
@@
 $EndComp
 $Comp
-L GND #PWR031
+L GND #PWR024
 U 1 1 5A4CF13E
 P 4800 2700
-F 0 "#PWR031" H 4800 2450 50  0001 C CNN
+F 0 "#PWR024" H 4800 2450 50  0001 C CNN
 F 1 "GND" H 4800 2550 50  0000 C CNN
 F 2 "" H 4800 2700 50  0000 C CNN
@@
 $EndComp
 $Comp
-L GND #PWR032
+L GND #PWR025
 U 1 1 5A4CF1BC
 P 5800 2700
-F 0 "#PWR032" H 5800 2450 50  0001 C CNN
+F 0 "#PWR025" H 5800 2450 50  0001 C CNN
 F 1 "GND" H 5800 2550 50  0000 C CNN
 F 2 "" H 5800 2700 50  0000 C CNN
@@
 $EndComp
 $Comp
-L GND #PWR033
+L GND #PWR026
 U 1 1 5A4CF1EB
 P 6650 2700
-F 0 "#PWR033" H 6650 2450 50  0001 C CNN
+F 0 "#PWR026" H 6650 2450 50  0001 C CNN
 F 1 "GND" H 6650 2550 50  0000 C CNN
 F 2 "" H 6650 2700 50  0000 C CNN
@@
 $EndComp
 $Comp
-L GND #PWR034
+L GND #PWR027
 U 1 1 5A4CF21A
 P 7300 2700
-F 0 "#PWR034" H 7300 2450 50  0001 C CNN
+F 0 "#PWR027" H 7300 2450 50  0001 C CNN
 F 1 "GND" H 7300 2550 50  0000 C CNN
 F 2 "" H 7300 2700 50  0000 C CNN
@@
 $EndComp
 $Comp
-L GND #PWR035
+L GND #PWR028
 U 1 1 5A4CF249
 P 8500 2700
-F 0 "#PWR035" H 8500 2450 50  0001 C CNN
+F 0 "#PWR028" H 8500 2450 50  0001 C CNN
 F 1 "GND" H 8500 2550 50  0000 C CNN
 F 2 "" H 8500 2700 50  0000 C CNN
@@
 $EndComp
 $Comp
-L GND #PWR036
+L GND #PWR029
 U 1 1 5A4CF278
 P 9100 2700
-F 0 "#PWR036" H 9100 2450 50  0001 C CNN
+F 0 "#PWR029" H 9100 2450 50  0001 C CNN
 F 1 "GND" H 9100 2550 50  0000 C CNN
 F 2 "" H 9100 2700 50  0000 C CNN
@@
 Wire Wire Line
 	7300 2700 7300 2650
-Wire Wire Line
-	4800 1250 4800 1700
 Wire Wire Line
 	4800 1400 4950 1400
@@
 	7300 1700 7350 1700
 $Comp
-L +3.3VADC #PWR037
-U 1 1 5A7450C0
-P 4800 1250
-F 0 "#PWR037" H 4950 1200 50  0001 C CNN
-F 1 "+3.3VADC" H 4800 1350 50  0000 C CNN
-F 2 "" H 4800 1250 50  0001 C CNN
-F 3 "" H 4800 1250 50  0001 C CNN
-	1    4800 1250
-	1    0    0    -1
-$EndComp
-$Comp
 L POT RV1
 U 1 1 5A746D57
 P 7500 1700
-F 0 "RV1" V 7325 1700 50  0000 C CNN
-F 1 "200k" V 7400 1700 50  0000 C CNN
+F 0 "RV1" V 7400 1700 50  0000 C CNN
+F 1 "200k" V 7500 1700 50  0000 C CNN
 F 2 "Zusatzteile:ST4ETA" H 7500 1700 50  0001 C CNN
 F 3 "" H 7500 1700 50  0001 C CNN
@@
 	7500 1850 7300 1850
 Connection ~ 7300 1850
+Connection ~ 6350 1400
+Connection ~ 6950 1400
+Connection ~ 8500 1400
+Connection ~ 9100 1400
+Connection ~ 6100 2000
+Wire Wire Line
+	4800 1250 4800 1700
+$Comp
+L +5V #PWR030
+U 1 1 5A793374
+P 4800 1250
+F 0 "#PWR030" H 4800 1100 50  0001 C CNN
+F 1 "+5V" H 4800 1390 50  0000 C CNN
+F 2 "" H 4800 1250 50  0001 C CNN
+F 3 "" H 4800 1250 50  0001 C CNN
+	1    4800 1250
+	1    0    0    -1
+$EndComp
 $EndSCHEMATC

Commit message: Layout
Parts:
- added R17: 0, kicad-libraries:R0603F, symbol R
Connections:
- net +5V: now also R17.1; no longer C5.1, L1.1
- new net: C5.1, L1.1, R17.2
Changed lines of the file:
@@
 Connection ~ 9100 1400
 Connection ~ 6100 2000
-Wire Wire Line
-	4800 1250 4800 1700
 $Comp
 L +5V #PWR031
 U 1 1 5A793374
-P 4800 1250
-F 0 "#PWR031" H 4800 1100 50  0001 C CNN
-F 1 "+5V" H 4800 1390 50  0000 C CNN
-F 2 "" H 4800 1250 50  0001 C CNN
-F 3 "" H 4800 1250 50  0001 C CNN
-	1    4800 1250
+P 4800 800
+F 0 "#PWR031" H 4800 650 50  0001 C CNN
+F 1 "+5V" H 4800 940 50  0000 C CNN
+F 2 "" H 4800 800 50  0001 C CNN
+F 3 "" H 4800 800 50  0001 C CNN
+	1    4800 800
 	1    0    0    -1
 $EndComp
+$Comp
+L R R17
+U 1 1 5A795820
+P 4800 1100
+F 0 "R17" V 4880 1100 50  0000 C CNN
+F 1 "0" V 4800 1100 50  0000 C CNN
+F 2 "kicad-libraries:R0603F" H 4800 1100 60  0000 C CNN
+F 3 "" H 4800 1100 60  0000 C CNN
+	1    4800 1100
+	1    0    0    -1
+$EndComp
+Wire Wire Line
+	4800 1350 4800 1700
+Wire Wire Line
+	4800 850  4800 800
 $EndSCHEMATC
