File: hardware/Prototyp/Schaltplan_Ultraschallsensor/_saved_sensor.sch (KiCad schematic (older format))
At the start: 18 parts, among them U2 TLC272, U5 DRILL, U6 DRILL

Commit message: software
Parts:
- C12: value 40pF -> 100nF
Connections:
- net Sensor- is gone; now on net GND: C10.2, C11.2, D2.1 (A), R11.2, R5.2, R9.2
- net GND: now also R4.2
- net Sensor+: now also R4.1
Other:
- moved on the sheet: C?, R4
Changed lines of the file:
@@
 L R R4
 U 1 1 5A4CEE2C
-P 1950 2400
-F 0 "R4" V 2030 2400 50  0000 C CNN
-F 1 "20k" V 1950 2400 50  0000 C CNN
-F 2 "kicad-libraries:R0603F" V 1880 2400 50  0001 C CNN
-F 3 "" H 1950 2400 50  0000 C CNN
-	1    1950 2400
+P 2050 2550
+F 0 "R4" V 2130 2550 50  0000 C CNN
+F 1 "20k" V 2050 2550 50  0000 C CNN
+F 2 "kicad-libraries:R0603F" V 1980 2550 50  0001 C CNN
+F 3 "" H 2050 2550 50  0000 C CNN
+	1    2050 2550
 	1    0    0    -1
 $EndComp
@@
 P 2400 1900
 F 0 "C12" H 2425 2000 50  0000 L CNN
-F 1 "40pF" H 2425 1800 50  0000 L CNN
+F 1 "100nF" H 2425 1800 50  0000 L CNN
 F 2 "kicad-libraries:C0603F" H 2438 1750 50  0001 C CNN
 F 3 "" H 2400 1900 50  0000 C CNN
@@
 L C C?
 U 1 1 5A957E2B
-P 2250 2400
-F 0 "C?" H 2300 2500 50  0000 L CNN
-F 1 "C" H 2300 2300 50  0000 L CNN
-F 2 "" H 2250 2400 60  0000 C CNN
-F 3 "" H 2250 2400 60  0000 C CNN
-	1    2250 2400
-	1    0    0    -1
-$EndComp
+P 1100 3200
+F 0 "C?" H 1150 3300 50  0000 L CNN
+F 1 "C" H 1150 3100 50  0000 L CNN
+F 2 "" H 1100 3200 60  0000 C CNN
+F 3 "" H 1100 3200 60  0000 C CNN
+	1    1100 3200
+	1    0    0    -1
+$EndComp
+Wire Wire Line
+	2050 1900 2050 2300
+Connection ~ 2050 1900
+Wire Wire Line
+	2050 2800 2050 3850
+Connection ~ 2050 3850
+Wire Wire Line
+	2200 3850 2200 4100
 $EndSCHEMATC

Commit message: doku
Parts:
- C12: value 100nF -> 40pF
Connections:
- net GND: no longer R4.2
- net Sensor+: no longer R4.1
Other:
- moved on the sheet: C?, R4
Changed lines of the file:
@@
 EESchema Schematic File Version 2
+LIBS:tinkerforge
 LIBS:meine
 LIBS:power
@@
 L R R4
 U 1 1 5A4CEE2C
-P 2050 2550
-F 0 "R4" V 2130 2550 50  0000 C CNN
-F 1 "20k" V 2050 2550 50  0000 C CNN
-F 2 "kicad-libraries:R0603F" V 1980 2550 50  0001 C CNN
-F 3 "" H 2050 2550 50  0000 C CNN
-	1    2050 2550
+P 1950 2400
+F 0 "R4" V 2030 2400 50  0000 C CNN
+F 1 "20k" V 1950 2400 50  0000 C CNN
+F 2 "kicad-libraries:R0603F" V 1880 2400 50  0001 C CNN
+F 3 "" H 1950 2400 50  0000 C CNN
+	1    1950 2400
 	1    0    0    -1
 $EndComp
@@
 P 2400 1900
 F 0 "C12" H 2425 2000 50  0000 L CNN
-F 1 "100nF" H 2425 1800 50  0000 L CNN
+F 1 "40pF" H 2425 1800 50  0000 L CNN
 F 2 "kicad-libraries:C0603F" H 2438 1750 50  0001 C CNN
 F 3 "" H 2400 1900 50  0000 C CNN
@@
 F 0 "C16" H 1650 1500 50  0000 L CNN
 F 1 "100nF" H 1650 1300 50  0000 L CNN
-F 2 "kicad-libraries:C0603F" H 1600 1400 60  0000 C CNN
+F 2 "kicad-libraries:C0603F" H 1600 1400 60  0001 C CNN
 F 3 "" H 1600 1400 60  0000 C CNN
 	1    1600 1400
@@
 L C C?
 U 1 1 5A957E2B
-P 1100 3200
-F 0 "C?" H 1150 3300 50  0000 L CNN
-F 1 "C" H 1150 3100 50  0000 L CNN
-F 2 "" H 1100 3200 60  0000 C CNN
-F 3 "" H 1100 3200 60  0000 C CNN
-	1    1100 3200
-	1    0    0    -1
-$EndComp
-Wire Wire Line
-	2050 1900 2050 2300
-Connection ~ 2050 1900
-Wire Wire Line
-	2050 2800 2050 3850
-Connection ~ 2050 3850
+P 2250 2400
+F 0 "C?" H 2300 2500 50  0000 L CNN
+F 1 "C" H 2300 2300 50  0000 L CNN
+F 2 "" H 2250 2400 60  0000 C CNN
+F 3 "" H 2250 2400 60  0000 C CNN
+	1    2250 2400
+	1    0    0    -1
+$EndComp
 Wire Wire Line
 	2200 3850 2200 4100
