File: hardware/Prototyp/Board_V2/Ultraschallsensor.kicad_pcb (KiCad board)
At the start: 2 copper layers, 49.5 x 38.1 mm, 63 parts, among them J1 Conn_01x02, P0 CON-SENSOR2, P1 CONN_01X01, P2 MP-PWM-2, P3 MP-Sensor-, P4 MP-Sensor+, P5 MP-PWM-1, P6 MP-PWM-2, P7 MP-OPV-AUS, P8 MP-OPV-ZK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

Commit message: HardwareV2b
Parts:
- removed RP2: R_PACK4, kicad-libraries:0603X4
- added R23: 10k, kicad-libraries:R0603F, F.Cu at (150.7, 79.0)
- added R24: 10k, kicad-libraries:R0603F, F.Cu at (154.6, 77.8)
- Q3: value MOSFET_N_P_CH -> DMG6602SVT-7DICT-ND
Routing:
- net Net-(RP1-Pad4): track 20.8 -> 18.0 mm
- net Net-(RP1-Pad3): track 14.0 -> 11.4 mm
- net Net-(RP1-Pad2): track 13.3 -> 11.2 mm, vias 2 -> 0
- net GND: track 64.2 -> 62.7 mm, vias 46 -> 44
- net PWM-2-OUT: track 12.8 -> 14.1 mm
- net PWM-1-OUT: track 12.0 -> 12.6 mm

Commit message: Update_Hardware
Routing:
- net GND: track 62.7 -> 67.8 mm, vias 44 -> 50

Commit message: set clearance to 0
Other:
- rule pad_to_mask_clearance: 0.2 -> 0
Changed lines of the file:
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@@
-(kicad_pcb (version 4) (host pcbnew 4.0.7-e2-6376~58~ubuntu16.04.1)
+(kicad_pcb (version 4) (host pcbnew 4.0.7-e2-6376~58~ubuntu17.04.1)
   (general
     (links 131)
@@
   )
   (setup
-    (last_trace_width 0.8)
+    (last_trace_width 0.2)
     (user_trace_width 0.25)
     (user_trace_width 0.3)
@@
     (pad_size 1.524 1.524)
     (pad_drill 0.762)
-    (pad_to_mask_clearance 0.2)
-    (aux_axis_origin 0 0)
+    (pad_to_mask_clearance 0)
+    (aux_axis_origin 174 88.9)
+    (grid_origin 174 88.9)
     (visible_elements FFFFFF7F)
     (pcbplotparams
-      (layerselection 0x00030_80000001)
+      (layerselection 0x010f8_80000001)
       (usegerberextensions false)
       (excludeedgelayer true)
@@
       (outputformat 1)
       (mirror false)
-      (drillshape 1)
+      (drillshape 0)
       (scaleselection 1)
-      (outputdirectory ""))
+      (outputdirectory pcb))
   )
   (net 0 "")
@@
   (segment (start 163.068 56.88076) (end 163.068 58.281) (width 1) (layer F.Cu) (net 1))
   (segment (start 163.068 58.281) (end 163.08 58.293) (width 1) (layer F.Cu) (net 1))
-  (segment (start 163.068 54.87924) (end 163.068 54.102) (width 0.6) (layer F.Cu) (net 2) (status 400000))
+  (segment (start 163.068 54.87924) (end 163.068 54.102) (width 0.6) (layer F.Cu) (net 2))
   (via (at 163.322 53.848) (size 0.7) (drill 0.25) (layers F.Cu B.Cu) (net 2))
   (segment (start 163.068 54.102) (end 163.322 53.848) (width 0.6) (layer F.Cu) (net 2))
-  (segment (start 163.068 54.87924) (end 163.068 54.2925) (width 0.6) (layer F.Cu) (net 2) (status 400000))
+  (segment (start 163.068 54.87924) (end 163.068 54.2925) (width 0.6) (layer F.Cu) (net 2))
   (via (at 162.6235 53.848) (size 0.7) (drill 0.25) (layers F.Cu B.Cu) (net 2))
   (segment (start 163.068 54.2925) (end 162.6235 53.848) (width 0.6) (layer F.Cu) (net 2))
-  (segment (start 161.40938 82.1055) (end 161.9885 82.1055) (width 0.7) (layer F.Cu) (net 2) (status 400000))
+  (segment (start 161.40938 82.1055) (end 161.9885 82.1055) (width 0.7) (layer F.Cu) (net 2))
   (via (at 162.433 82.55) (size 0.7) (drill 0.25) (layers F.Cu B.Cu) (net 2))
   (segment (start 161.9885 82.1055) (end 162.433 82.55) (width 0.7) (layer F.Cu) (net 2))
-  (segment (start 161.40938 82.1055) (end 162.2425 82.1055) (width 0.7) (layer F.Cu) (net 2) (status 400000))
+  (segment (start 161.40938 82.1055) (end 162.2425 82.1055) (width 0.7) (layer F.Cu) (net 2))
   (via (at 162.433 81.915) (size 0.7) (drill 0.25) (layers F.Cu B.Cu) (net 2))
   (segment (start 162.2425 82.1055) (end 162.433 81.915) (width 0.7) (layer F.Cu) (net 2))
@@
   (via (at 157.099 55.9435) (size 0.7) (drill 0.25) (layers F.Cu B.Cu) (net 2))
   (segment (start 156.551 56.4915) (end 157.099 55.9435) (width 0.7) (layer F.Cu) (net 2))
-  (segment (start 156.551 57.559) (end 156.551 56.5785) (width 0.7) (layer F.Cu) (net 2) (status 400000))
+  (segment (start 156.551 57.559) (end 156.551 56.5785) (width 0.7) (layer F.Cu) (net 2))
   (segment (start 156.551 56.5785) (end 156.551 56.094) (width 0.7) (layer F.Cu) (net 2))
   (via (at 156.4005 55.9435) (size 0.7) (drill 0.25) (layers F.Cu B.Cu) (net 2))
   (segment (start 156.551 56.094) (end 156.4005 55.9435) (width 0.7) (layer F.Cu) (net 2))
-  (segment (start 156.551 57.559) (end 156.551 58.888) (width 0.7) (layer F.Cu) (net 2) (status 400000))
+  (segment (start 156.551 57.559) (end 156.551 58.888) (width 0.7) (layer F.Cu) (net 2))
   (via (at 156.972 59.309) (size 0.7) (drill 0.25) (layers F.Cu B.Cu) (net 2))
   (segment (start 156.551 58.888) (end 156.972 59.309) (width 0.7) (layer F.Cu) (net 2))
-  (segment (start 156.551 57.559) (end 156.551 59.0315) (width 0.7) (layer F.Cu) (net 2) (status 400000))
+  (segment (start 156.551 57.559) (end 156.551 59.0315) (width 0.7) (layer F.Cu) (net 2))
   (via (at 156.2735 59.309) (size 0.7) (drill 0.25) (layers F.Cu B.Cu) (net 2))
   (segment (start 156.551 59.0315) (end 156.2735 59.309) (width 0.7) (layer F.Cu) (net 2))
@@
   (segment (start 133.235 71.12) (end 133.235 68.326) (width 0.25) (layer F.Cu) (net 10))
   (segment (start 133.03758 71.31742) (end 133.235 71.12) (width 0.3) (layer F.Cu) (net 10))
-  (segment (start 156.44876 70.739) (end 156.44876 74.53376) (width 0.8) (layer F.Cu) (net 11) (status 400000))
-  (segment (start 160.8485 76.965) (end 160.8485 78.1685) (width 0.8) (layer F.Cu) (net 11) (status 800000))
+  (segment (start 156.44876 70.739) (end 156.44876 74.53376) (width 0.8) (layer F.Cu) (net 11))
+  (segment (start 160.8485 76.965) (end 160.8485 78.1685) (width 0.8) (layer F.Cu) (net 11))
   (segment (start 160.2105 76.327) (end 160.8485 76.965) (width 0.8) (layer F.Cu) (net 11))
   (segment (start 158.242 76.327) (end 160.2105 76.327) (width 0.8) (layer F.Cu) (net 11))
@@
   (segment (start 158.115 81.15554) (end 157.86354 81.15554) (width 0.7) (layer F.Cu) (net 23))
   (segment (start 157.86354 81.15554) (end 157.0355 80.3275) (width 0.7) (layer F.Cu) (net 23))
-  (segment (start 152.70988 75.53452) (end 153.63698 75.53452) (width 0.25) (layer F.Cu) (net 24) (status 400000))
-  (segment (start 165.02888 70.61962) (end 165.02888 66.98996) (width 0.25) (layer F.Cu) (net 24) (status 800000))
+  (segment (start 152.70988 75.53452) (end 153.63698 75.53452) (width 0.25) (layer F.Cu) (net 24))
+  (segment (start 165.02888 70.61962) (end 165.02888 66.98996) (width 0.25) (layer F.Cu) (net 24))
   (segment (start 163.5125 72.136) (end 165.02888 70.61962) (width 0.25) (layer F.Cu) (net 24))
   (via (at 163.5125 72.136) (size 0.7) (drill 0.25) (layers F.Cu B.Cu) (net 24))

Commit message: update documentation
Parts:
- moved RV1 0.17 mm to (138.7, 73.7)
Changed lines of the file:
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@@
-(kicad_pcb (version 4) (host pcbnew 4.0.7-e2-6376~58~ubuntu17.04.1)
+(kicad_pcb (version 4) (host pcbnew 4.0.7-e2-6376~58~ubuntu16.04.1)
   (general
     (links 131)
@@
   (module kicad-libraries:QFN48-EP2 (layer F.Cu)
     (at 149.098 73.787 90)
-    (fp_text reference U3 (at 0 0 90) (layer F.SilkS)
-      (effects (font (size 0.29972 0.29972) (thickness 0.0762)))
-    )
-    (fp_text value XMC1XXX48 (at 0 -0.7 90) (layer F.SilkS)
-      (effects (font (size 0.29972 0.29972) (thickness 0.0762)))
+    (fp_text reference U3 (at 1.651 -2.276 90) (layer F.Fab)
+      (effects (font (size 0.29972 0.29972) (thickness 0.07493)))
+    )
+    (fp_text value XMC1XXX48 (at -0.381 -2.276 90) (layer F.Fab)
+      (effects (font (size 0.29972 0.29972) (thickness 0.07493)))
     )
     (fp_circle (center -2.5 2.6) (end -2.4 2.8) (layer F.Fab) (width 0.05))
@@
   (module kicad-libraries:CON-SENSOR2 (layer F.Cu)
     (at 154.051 52.959 180)
-    (fp_text reference P0 (at 0 -2.85 180) (layer F.Fab)
+    (fp_text reference P0 (at 0.117 -2.159 180) (layer F.Fab)
       (effects (font (size 0.3 0.3) (thickness 0.075)))
     )
@@
       (rotate (xyz 0 0 0))
     )
-  )
-  (module kicad-libraries:ST4 (layer F.Cu)
-    (at 138.811 73.533 270)
-    (fp_text reference RV1 (at 3.8735 -0.4445 270) (layer F.Fab)
-      (effects (font (size 1 1) (thickness 0.15)))
-    )
-    (fp_text value 50k (at 0 0 270) (layer F.Fab)
-      (effects (font (size 1 1) (thickness 0.15)))
-    )
-    (fp_line (start 2.794 1.651) (end 2.794 3.175) (layer F.CrtYd) (width 0.1))
-    (fp_line (start 2.794 3.175) (end -2.794 3.175) (layer F.CrtYd) (width 0.1))
-    (fp_line (start -2.794 3.175) (end -2.794 2.54) (layer F.CrtYd) (width 0.1))
-    (fp_line (start 2.794 -3.175) (end -2.794 -3.175) (layer F.CrtYd) (width 0.1))
-    (fp_line (start -2.794 -3.175) (end -2.794 2.54) (layer F.CrtYd) (width 0.1))
-    (fp_line (start 2.794 -3.175) (end 2.794 1.651) (layer F.CrtYd) (width 0.1))
-    (fp_line (start -2.159 2.286) (end -2.413 2.286) (layer F.SilkS) (width 0.15))
-    (fp_line (start -2.413 2.286) (end -2.413 -2.286) (layer F.SilkS) (width 0.15))
-    (fp_line (start -2.413 -2.286) (end -1.143 -2.286) (layer F.SilkS) (width 0.15))
-    (fp_line (start 1.143 -2.286) (end 2.413 -2.286) (layer F.SilkS) (width 0.15))
-    (fp_line (start 2.413 -2.286) (end 2.413 2.286) (layer F.SilkS) (width 0.15))
-    (fp_line (start 2.159 2.286) (end 2.413 2.286) (layer F.SilkS) (width 0.15))
-    (pad 1 smd rect (at 1.175 2 270) (size 1.6 2) (layers F.Cu F.Paste F.Mask)
-      (net 63 "Net-(R6-Pad1)"))
-    (pad 3 smd rect (at -1.175 2 270) (size 1.6 2) (layers F.Cu F.Paste F.Mask)
-      (net 62 "Net-(P8-Pad1)"))
-    (pad 2 smd rect (at 0 -2 270) (size 2 2) (layers F.Cu F.Paste F.Mask)
-      (net 63 "Net-(R6-Pad1)"))
-  )
-  (module kicad-libraries:ST4 (layer F.Cu)
-    (at 161.544 72.39 180)
-    (fp_text reference RV2 (at -0.762 4.064 180) (layer F.SilkS)
-      (effects (font (size 1 1) (thickness 0.15)))
-    )
-    (fp_text value 200k (at 0 0 180) (layer F.Fab)
-      (effects (font (size 1 1) (thickness 0.15)))
-    )
-    (fp_line (start 2.794 1.651) (end 2.794 3.175) (layer F.CrtYd) (width 0.1))
-    (fp_line (start 2.794 3.175) (end -2.794 3.175) (layer F.CrtYd) (width 0.1))
-    (fp_line (start -2.794 3.175) (end -2.794 2.54) (layer F.CrtYd) (width 0.1))
-    (fp_line (start 2.794 -3.175) (end -2.794 -3.175) (layer F.CrtYd) (width 0.1))
-    (fp_line (start -2.794 -3.175) (end -2.794 2.54) (layer F.CrtYd) (width 0.1))
-    (fp_line (start 2.794 -3.175) (end 2.794 1.651) (layer F.CrtYd) (width 0.1))
-    (fp_line (start -2.159 2.286) (end -2.413 2.286) (layer F.SilkS) (width 0.15))
-    (fp_line (start -2.413 2.286) (end -2.413 -2.286) (layer F.SilkS) (width 0.15))
-    (fp_line (start -2.413 -2.286) (end -1.143 -2.286) (layer F.SilkS) (width 0.15))
-    (fp_line (start 1.143 -2.286) (end 2.413 -2.286) (layer F.SilkS) (width 0.15))
-    (fp_line (start 2.413 -2.286) (end 2.413 2.286) (layer F.SilkS) (width 0.15))
-    (fp_line (start 2.159 2.286) (end 2.413 2.286) (layer F.SilkS) (width 0.15))
-    (pad 1 smd rect (at 1.175 2 180) (size 1.6 2) (layers F.Cu F.Paste F.Mask)
-      (net 64 "Net-(R10-Pad2)"))
-    (pad 3 smd rect (at -1.175 2 180) (size 1.6 2) (layers F.Cu F.Paste F.Mask)
-      (net 9 "Net-(C6-Pad2)"))
-    (pad 2 smd rect (at 0 -2 180) (size 2 2) (layers F.Cu F.Paste F.Mask)
-      (net 9 "Net-(C6-Pad2)"))
   )
   (module kicad-libraries:SOT23-6 (layer F.Cu)
@@
     )
   )
+  (module kicad-libraries:ST4 (layer F.Cu)
+    (at 138.694 73.66 270)
+    (fp_text reference RV1 (at -1.397 0.381 270) (layer F.Fab)
+      (effects (font (size 0.4 0.4) (thickness 0.1)))
+    )
+    (fp_text value 50k (at -1.651 -0.508 270) (layer F.Fab)
+      (effects (font (size 0.4 0.4) (thickness 0.1)))
+    )
+    (fp_line (start 2.794 1.651) (end 2.794 3.175) (layer F.CrtYd) (width 0.1))
+    (fp_line (start 2.794 3.175) (end -2.794 3.175) (layer F.CrtYd) (width 0.1))
+    (fp_line (start -2.794 3.175) (end -2.794 2.54) (layer F.CrtYd) (width 0.1))
+    (fp_line (start 2.794 -3.175) (end -2.794 -3.175) (layer F.CrtYd) (width 0.1))
+    (fp_line (start -2.794 -3.175) (end -2.794 2.54) (layer F.CrtYd) (width 0.1))
+    (fp_line (start 2.794 -3.175) (end 2.794 1.651) (layer F.CrtYd) (width 0.1))
+    (fp_line (start -2.159 2.286) (end -2.413 2.286) (layer F.Fab) (width 0.15))
+    (fp_line (start -2.413 2.286) (end -2.413 -2.286) (layer F.Fab) (width 0.15))
+    (fp_line (start -2.413 -2.286) (end -1.143 -2.286) (layer F.Fab) (width 0.15))
+    (fp_line (start 1.143 -2.286) (end 2.413 -2.286) (layer F.Fab) (width 0.15))
+    (fp_line (start 2.413 -2.286) (end 2.413 2.286) (layer F.Fab) (width 0.15))
+    (fp_line (start 2.159 2.286) (end 2.413 2.286) (layer F.Fab) (width 0.15))
+    (pad 1 smd rect (at 1.175 2 270) (size 1.6 2) (layers F.Cu F.Paste F.Mask)
+      (net 63 "Net-(R6-Pad1)"))
+    (pad 3 smd rect (at -1.175 2 270) (size 1.6 2) (layers F.Cu F.Paste F.Mask)
+      (net 62 "Net-(P8-Pad1)"))
+    (pad 2 smd rect (at 0 -2 270) (size 2 2) (layers F.Cu F.Paste F.Mask)
+      (net 63 "Net-(R6-Pad1)"))
+  )
+  (module kicad-libraries:ST4 (layer F.Cu)
+    (at 161.554 72.39 180)
+    (fp_text reference RV2 (at 1.778 -0.508 180) (layer F.Fab)
+      (effects (font (size 0.4 0.4) (thickness 0.1)))
+    )
+    (fp_text value 200k (at -1.651 -0.508 180) (layer F.Fab)
+      (effects (font (size 0.4 0.4) (thickness 0.1)))
+    )
+    (fp_line (start 2.794 1.651) (end 2.794 3.175) (layer F.CrtYd) (width 0.1))
+    (fp_line (start 2.794 3.175) (end -2.794 3.175) (layer F.CrtYd) (width 0.1))
+    (fp_line (start -2.794 3.175) (end -2.794 2.54) (layer F.CrtYd) (width 0.1))
+    (fp_line (start 2.794 -3.175) (end -2.794 -3.175) (layer F.CrtYd) (width 0.1))
+    (fp_line (start -2.794 -3.175) (end -2.794 2.54) (layer F.CrtYd) (width 0.1))
+    (fp_line (start 2.794 -3.175) (end 2.794 1.651) (layer F.CrtYd) (width 0.1))
+    (fp_line (start -2.159 2.286) (end -2.413 2.286) (layer F.Fab) (width 0.15))
+    (fp_line (start -2.413 2.286) (end -2.413 -2.286) (layer F.Fab) (width 0.15))
+    (fp_line (start -2.413 -2.286) (end -1.143 -2.286) (layer F.Fab) (width 0.15))
+    (fp_line (start 1.143 -2.286) (end 2.413 -2.286) (layer F.Fab) (width 0.15))
+    (fp_line (start 2.413 -2.286) (end 2.413 2.286) (layer F.Fab) (width 0.15))
+    (fp_line (start 2.159 2.286) (end 2.413 2.286) (layer F.Fab) (width 0.15))
+    (pad 1 smd rect (at 1.175 2 180) (size 1.6 2) (layers F.Cu F.Paste F.Mask)
+      (net 64 "Net-(R10-Pad2)"))
+    (pad 3 smd rect (at -1.175 2 180) (size 1.6 2) (layers F.Cu F.Paste F.Mask)
+      (net 9 "Net-(C6-Pad2)"))
+    (pad 2 smd rect (at 0 -2 180) (size 2 2) (layers F.Cu F.Paste F.Mask)
+      (net 9 "Net-(C6-Pad2)"))
+  )
   (gr_line (start 173.99 81.28) (end 166.37 88.9) (angle 90) (layer Edge.Cuts) (width 0.15))

Commit message: Korrektur pcb
Parts:
- P2: value MP-PWM-2 -> MP-GND
- moved P2 0.83 mm to (148.0, 85.6)
- moved P1 0.66 mm to (144.1, 85.6)
Connections:
- Q3 pad 2: Net-(LS1-Pad1) -> +UA
- Q3 pad 4: +UA -> Net-(LS1-Pad1)
Routing:
- net Net-(LS1-Pad1): track 31.9 -> 39.6 mm, vias 2 -> 0
- net +UA: track 30.1 -> 31.9 mm
- net Net-(P1-Pad1): track 14.4 -> 13.9 mm
Changed lines of the file:
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@@
     (thickness 1.6)
     (drawings 8)
-    (tracks 528)
+    (tracks 525)
     (zones 0)
     (modules 64)
@@
   )
   (module kicad-libraries:CONN_1 (layer F.Cu)
-    (at 144.272 86.233)
+    (at 144.1 85.6)
     (fp_text reference P1 (at -0.09906 0.59944) (layer F.SilkS) hide
       (effects (font (size 0.127 0.127) (thickness 0.00254)))
@@
     (pad 1 thru_hole circle (at 0 0) (size 3.50012 3.50012) (drill 1.50114) (layers *.Cu *.Mask F.SilkS)
       (net 61 "Net-(P1-Pad1)") (clearance 0.14986))
-  )
-  (module kicad-libraries:CONN_1 (layer F.Cu)
-    (at 148.336 86.36)
-    (fp_text reference P2 (at -0.09906 0.59944) (layer F.SilkS) hide
-      (effects (font (size 0.127 0.127) (thickness 0.00254)))
-    )
-    (fp_text value MP-PWM-2 (at 0 -0.50038) (layer F.SilkS) hide
-      (effects (font (size 0.127 0.127) (thickness 0.00254)))
-    )
-    (pad 1 thru_hole circle (at 0 0) (size 3.50012 3.50012) (drill 1.50114) (layers *.Cu *.Mask F.SilkS)
-      (net 2 GND) (clearance 0.14986))
   )
   (module kicad-libraries:R0603F (layer B.Cu)
@@
       (net 23 "Net-(Q2-PadD)") (clearance 0.14986))
     (pad 2 smd rect (at 0 1.19888 270) (size 0.50038 0.8001) (layers F.Cu F.Paste F.Mask)
-      (net 57 "Net-(LS1-Pad1)") (clearance 0.14986))
+      (net 11 +UA) (clearance 0.14986))
     (pad 3 smd rect (at 0.94996 1.19888 270) (size 0.50038 0.8001) (layers F.Cu F.Paste F.Mask)
       (net 21 "Net-(Q1-PadD)") (clearance 0.14986))
@@
       (net 57 "Net-(LS1-Pad1)") (clearance 0.14986))
     (pad 4 smd rect (at 0.94996 -1.19888 270) (size 0.50038 0.8001) (layers F.Cu F.Paste F.Mask)
-      (net 11 +UA) (clearance 0.14986))
+      (net 57 "Net-(LS1-Pad1)") (clearance 0.14986))
     (pad 5 smd rect (at 0 -1.19888 270) (size 0.50038 0.8001) (layers F.Cu F.Paste F.Mask)
       (net 2 GND) (clearance 0.14986))
@@
     (pad 2 smd rect (at 0 -2 180) (size 2 2) (layers F.Cu F.Paste F.Mask)
       (net 9 "Net-(C6-Pad2)"))
+  )
+  (module kicad-libraries:CONN_1 (layer F.Cu)
+    (at 148 85.6)
+    (fp_text reference P2 (at -0.09906 0.59944) (layer F.SilkS) hide
+      (effects (font (size 0.127 0.127) (thickness 0.00254)))
+    )
+    (fp_text value MP-GND (at 0 -0.50038) (layer F.SilkS) hide
+      (effects (font (size 0.127 0.127) (thickness 0.00254)))
+    )
+    (pad 1 thru_hole circle (at 0 0) (size 3.50012 3.50012) (drill 1.50114) (layers *.Cu *.Mask F.SilkS)
+      (net 2 GND) (clearance 0.14986))
   )
   (gr_line (start 173.99 81.28) (end 166.37 88.9) (angle 90) (layer Edge.Cuts) (width 0.15))
@@
   (segment (start 133.235 71.12) (end 133.235 68.326) (width 0.25) (layer F.Cu) (net 10))
   (segment (start 133.03758 71.31742) (end 133.235 71.12) (width 0.3) (layer F.Cu) (net 10))
+  (segment (start 159.01162 82.1055) (end 159.6945 82.1055) (width 0.6) (layer F.Cu) (net 11))
+  (segment (start 160.2 80.338) (end 160.655 79.883) (width 0.6) (layer F.Cu) (net 11))
+  (segment (start 160.2 81.6) (end 160.2 80.338) (width 0.6) (layer F.Cu) (net 11))
+  (segment (start 159.6945 82.1055) (end 160.2 81.6) (width 0.6) (layer F.Cu) (net 11))
   (segment (start 156.44876 70.739) (end 156.44876 74.53376) (width 0.8) (layer F.Cu) (net 11))
   (segment (start 160.8485 76.965) (end 160.8485 78.1685) (width 0.8) (layer F.Cu) (net 11))
@@
   (segment (start 160.8485 78.1685) (end 160.8485 79.6895) (width 0.8) (layer F.Cu) (net 11))
   (segment (start 160.7215 86.0425) (end 160.7215 84.328) (width 0.8) (layer F.Cu) (net 11))
-  (segment (start 160.7215 84.328) (end 160.7215 83.74334) (width 0.8) (layer F.Cu) (net 11))
-  (segment (start 160.7215 83.74334) (end 161.40938 83.05546) (width 0.8) (layer F.Cu) (net 11))
   (segment (start 156.095 66.04) (end 156.095 70.38524) (width 0.8) (layer F.Cu) (net 11))
   (segment (start 156.095 70.38524) (end 156.44876 70.739) (width 0.7) (layer F.Cu) (net 11))
@@
   (segment (start 145.542 64.643) (end 148.463 61.722) (width 0.25) (layer F.Cu) (net 29))
   (segment (start 145.48612 71.03872) (end 145.48612 69.2785) (width 0.25) (layer F.Cu) (net 29))
-  (segment (start 159.01162 82.1055) (end 153.924 82.1055) (width 0.5) (layer F.Cu) (net 57))
-  (segment (start 140.1445 84.582) (end 138.799 84.582) (width 0.5) (layer F.Cu) (net 57))
-  (segment (start 140.5255 84.201) (end 140.1445 84.582) (width 0.5) (layer F.Cu) (net 57))
-  (via (at 140.5255 84.201) (size 0.55) (drill 0.25) (layers F.Cu B.Cu) (net 57))
-  (segment (start 140.9065 83.82) (end 140.5255 84.201) (width 0.5) (layer B.Cu) (net 57))
-  (segment (start 145.796 83.82) (end 140.9065 83.82) (width 0.5) (layer B.Cu) (net 57))
-  (segment (start 146.1135 84.1375) (end 145.796 83.82) (width 0.5) (layer B.Cu) (net 57))
-  (segment (start 153.035 84.1375) (end 146.1135 84.1375) (width 0.5) (layer B.Cu) (net 57))
-  (segment (start 153.7335 83.439) (end 153.035 84.1375) (width 0.5) (layer B.Cu) (net 57))
-  (segment (start 153.7335 82.296) (end 153.7335 83.439) (width 0.5) (layer B.Cu) (net 57))
-  (via (at 153.7335 82.296) (size 0.55) (drill 0.25) (layers F.Cu B.Cu) (net 57))
-  (segment (start 153.924 82.1055) (end 153.7335 82.296) (width 0.5) (layer F.Cu) (net 57))
+  (segment (start 138.938 86.487) (end 138.938 86.738) (width 0.6) (layer F.Cu) (net 57))
+  (segment (start 138.938 86.738) (end 140.1 87.9) (width 0.6) (layer F.Cu) (net 57))
+  (segment (start 162.3 84.334) (end 163.134 83.5) (width 0.6) (layer F.Cu) (net 57))
+  (segment (start 162.3 87.3) (end 162.3 84.334) (width 0.6) (layer F.Cu) (net 57))
+  (segment (start 161.7 87.9) (end 162.3 87.3) (width 0.6) (layer F.Cu) (net 57))
+  (segment (start 140.1 87.9) (end 161.7 87.9) (width 0.6) (layer F.Cu) (net 57))
+  (segment (start 161.40938 83.05546) (end 161.65546 83.05546) (width 0.6) (layer F.Cu) (net 57))
+  (segment (start 161.65546 83.05546) (end 162.1 83.5) (width 0.6) (layer F.Cu) (net 57))
+  (segment (start 162.1 83.5) (end 163.134 83.5) (width 0.6) (layer F.Cu) (net 57))
+  (segment (start 163.134 83.5) (end 164.719 81.915) (width 0.6) (layer F.Cu) (net 57))
   (segment (start 138.799 84.582) (end 138.799 86.348) (width 0.45) (layer F.Cu) (net 57))
   (segment (start 138.799 86.348) (end 138.938 86.487) (width 0.45) (layer F.Cu) (net 57))
@@
   (segment (start 163.95954 81.15554) (end 161.40938 81.15554) (width 0.5) (layer F.Cu) (net 57))
   (segment (start 164.719 81.915) (end 163.95954 81.15554) (width 0.5) (layer F.Cu) (net 57))
-  (segment (start 159.01162 82.1055) (end 159.7025 82.1055) (width 0.45) (layer F.Cu) (net 57))
-  (segment (start 160.65246 81.15554) (end 161.40938 81.15554) (width 0.45) (layer F.Cu) (net 57))
-  (segment (start 159.7025 82.1055) (end 160.65246 81.15554) (width 0.45) (layer F.Cu) (net 57))
   (segment (start 152.0063 60.512) (end 152.0063 60.0837) (width 0.3) (layer F.Cu) (net 58))
   (segment (start 154.051 58.801) (end 154.051 57.559) (width 0.3) (layer F.Cu) (net 58))
@@
   (segment (start 151.00808 59.55792) (end 151.551 59.015) (width 0.3) (layer F.Cu) (net 60))
   (segment (start 145.48612 75.53452) (end 144.68348 75.53452) (width 0.25) (layer F.Cu) (net 61))
-  (segment (start 141.7955 84.2645) (end 143.764 86.233) (width 0.25) (layer F.Cu) (net 61))
+  (segment (start 141.7955 84.2645) (end 143.592 85.6) (width 0.25) (layer F.Cu) (net 61) (status 20))
   (segment (start 141.7955 80.3275) (end 141.7955 84.2645) (width 0.25) (layer F.Cu) (net 61))
   (via (at 141.7955 80.3275) (size 0.55) (drill 0.25) (layers F.Cu B.Cu) (net 61))
@@
   (segment (start 144.0815 76.1365) (end 144.0815 76.3905) (width 0.25) (layer F.Cu) (net 61))
   (segment (start 144.68348 75.53452) (end 144.0815 76.1365) (width 0.25) (layer F.Cu) (net 61))
-  (segment (start 143.764 86.233) (end 144.272 86.233) (width 0.25) (layer F.Cu) (net 61))
-  (segment (start 143.891 86.233) (end 144.272 86.233) (width 0.3) (layer F.Cu) (net 61) (status 30))
+  (segment (start 143.592 85.6) (end 144.1 85.6) (width 0.25) (layer F.Cu) (net 61) (status 30))
+  (segment (start 143.719 85.6) (end 144.1 85.6) (width 0.3) (layer F.Cu) (net 61) (status 30))
   (segment (start 127.0635 81.3435) (end 127.0635 80.899) (width 0.3) (layer F.Cu) (net 62))
   (segment (start 127.0635 80.899) (end 129.159 78.8035) (width 0.3) (layer F.Cu) (net 62))
