File: hardware/Prototyp/Board_V2/Ultraschallsensor.sch (KiCad schematic (older format))
At the start: 54 parts

Commit message: HardwareV2
Parts:
- removed D? (x2): LED, kicad-libraries:D0603E, symbol LED
- removed P?: CONN_01X01, kicad-libraries:DEBUG_PAD, symbol CONN_01X01
- removed RP?: 1K, kicad-libraries:0603X4, symbol R_PACK4
- added P1: CONN_01X01, kicad-libraries:CONN_1, symbol CONN_01X01
- added P2: MP-PWM-2, kicad-libraries:CONN_1, symbol CONN_01X01
- added P3: MP-Sensor-, kicad-libraries:DEBUG_PAD, symbol CONN_01X01
- added P4: MP-Sensor+, kicad-libraries:DEBUG_PAD, symbol CONN_01X01
- added P5: MP-PWM-1, kicad-libraries:DEBUG_PAD, symbol CONN_01X01
- added P6: MP-PWM-2, kicad-libraries:DEBUG_PAD, symbol CONN_01X01
- added P7: MP-OPV-AUS, kicad-libraries:CONN_1, symbol CONN_01X01
- added P8: MP-OPV-ZK, kicad-libraries:CONN_1, symbol CONN_01X01
- added P9: MP-+UA, kicad-libraries:CONN_1, symbol CONN_01X01
- added Q1, Q2: MOSFET_N_CH, kicad-libraries:SOT23GDS, symbol MOSFET_N_CH
- added Q3: MOSFET_N_P_CH, kicad-libraries:SOT23-6, symbol MOSFET_N_P_CH
- added R14: 1k, kicad-libraries:R0603F, symbol R
- added R21, R22: 1k, kicad-libraries:1206E, symbol R
- added R30, R31: 0, kicad-libraries:R0603F, symbol R
- added RV1: 50k, kicad-libraries:ST4, symbol POT
- added RV2: 200k, kicad-libraries:ST4, symbol POT
- D2: renamed from D?; footprint (none) -> kicad-libraries:SOD-123
- LS1: renamed from LS?; footprint (none) -> kicad-libraries:PIN_ARRAY_2X1
- R10: renamed from R?; value R -> 20K
- R6: renamed from R?; value R -> 20k
- U3: renamed from U?; footprint (none) -> kicad-libraries:QFN48-EP2
- gave numbers to parts that had none: 40
Connections:
- net Sensor- is gone; now on net GND: C5.2, C9.2, D1.1 (A), LS1.2, R1.2, R11.2, R3.2, R9.2
- net +3V3: now also U3.18 (VDD), U3.19 (VDDP), U3.27 (VDDP), U3.38 (VDDP), R14.2; no longer U3.18 (VDD), U3.19 (VDDP), U3.27 (VDDP), U3.38 (VDDP)
- net +UA: now also P9.1 (P1), Q3.4 (D), R21.1, R22.1
- net GND: now also U3.17 (VSS), U3.37 (VSSP), U3.EP (VSSP), P2.1 (P1), P3.1 (P1), Q1.S, Q2.S, Q3.5 (S); no longer U3.17 (VSS), U3.37 (VSSP), U3.EP (VSSP)
- net MP-OPV-Aus: now also U3.12 (P2.9_AI), P7.1 (P1), R30.1
- net SHDN: now also U3.3 (P2.0_AIO)
- net Sensor+: now also R31.1; no longer LS1.1
- net at C6.2, R7.1, U2.3 (FB): now also RV2.3; no longer R10.2
- net at J1.2 (Pin_2): now also U3.36 (P0.7_IO); no longer U3.36 (P0.7_IO)
- net at C15.1, X1.2: now also U3.41 (P0.10_IO/XTAL1); no longer U3.41 (P0.10_IO/XTAL1)
- net at C16.1, X1.1: now also U3.42 (P0.11_IO/XTAL2); no longer U3.42 (P0.11_IO/XTAL2)
- net at D3.2 (K): now also U3.13 (P2.10/AIO); no longer U3.13 (P2.10/AIO)
- net at D3.1 (A): now also R14.1
- net MP-OPV-ZK: no longer names the net of U1.1 (OUT), U1.5 (IN+)
- net MP-OPV-ZK: now also P8.1 (P1), R30.2; no longer R6.1
- new net: R6.1, RV1.2, RV1.3
- new net: R10.2, RV2.2
- new net: P1.1 (P1), U3.34 (P0.5_IO)
- new net: LS1.1, P4.1 (P1), Q3.2 (S), Q3.6 (D), R31.2
- new net: Q1.D, Q3.3 (G), R22.2
- new net: Q2.D, Q3.1 (G), R21.2
- new net PWM-1-OUT: P5.1 (P1), Q1.G, U3.47 (P4.4_IO)
- new net PWM-2-OUT: P6.1 (P1), Q2.G, U3.1 (P4.6_IO)
- no-connect marks 32 -> 30
Other:
- moved on the sheet: C12, C13, D3, L3, LS1, R10

Commit message: HardwareV2b
Parts:
- removed RP2: R_PACK4, kicad-libraries:0603X4, symbol R_PACK4
- added R23, R24: 10k, kicad-libraries:R0603F, symbol R
- Q3: value MOSFET_N_P_CH -> DMG6602SVT-7DICT-ND
Connections:
- net GND: now also R23.2, R24.2
- net PWM-1-OUT: now also R23.1
- net PWM-2-OUT: now also R24.1
- no-connect marks 30 -> 29
Changed lines of the file:
@@
 Text GLabel 950  1250 0    60   Input ~ 0
 Sensor+
-Text GLabel 950  2850 0    60   Input ~ 0
-Sensor-
 $Comp
 L ZENER D1
@@
 	1000 1800 1000 2850
 Wire Wire Line
-	950  2850 4150 2850
-Wire Wire Line
-	1500 2850 1500 1800
+	1500 1800 1500 2900
 Connection ~ 1000 2850
 Wire Wire Line
@@
 Connection ~ 2800 1400
 Wire Wire Line
-	1650 1700 1650 2850
+	1650 2850 1650 1700
 Connection ~ 1650 2850
 Wire Wire Line
@@
 	-1   0    0    1
 $EndComp
-$Comp
-L R_PACK4 RP2
-U 1 1 5A946A44
-P 5950 7400
-F 0 "RP2" H 5950 7850 50  0000 C CNN
-F 1 "R_PACK4" H 5950 7350 50  0000 C CNN
-F 2 "kicad-libraries:0603X4" H 5950 7400 50  0001 C CNN
-F 3 "" H 5950 7400 50  0000 C CNN
-	1    5950 7400
-	0    1    1    0
-$EndComp
 Wire Wire Line
 	4900 6800 5000 6800
@@
 	5700 7150 6350 7150
 Wire Wire Line
-	6300 7200 6300 6650
-Connection ~ 6300 6650
-Wire Wire Line
-	6200 7200 6200 6750
-Connection ~ 6200 6750
-Wire Wire Line
-	6100 7200 6100 6850
-Connection ~ 6100 6850
-Wire Wire Line
-	6000 7650 6000 7600
-Wire Wire Line
-	4550 7650 6300 7650
-Wire Wire Line
-	6300 7650 6300 7600
-Wire Wire Line
-	6200 7650 6200 7600
-Connection ~ 6200 7650
-Wire Wire Line
-	6100 7650 6100 7600
-Connection ~ 6100 7650
+	4550 7650 4950 7650
 $Comp
 L C C14
@@
 Connection ~ 4950 7100
 Wire Wire Line
-	4950 7650 4950 7550
-Connection ~ 6000 7650
+	4950 7550 4950 7700
 Wire Wire Line
 	4550 7650 4550 7250
@@
 L GND #PWR06
 U 1 1 5A948103
-P 5500 7700
-F 0 "#PWR06" H 5500 7700 30  0001 C CNN
-F 1 "GND" H 5500 7630 30  0001 C CNN
-F 2 "" H 5500 7700 60  0000 C CNN
-F 3 "" H 5500 7700 60  0000 C CNN
-	1    5500 7700
-	1    0    0    -1
-$EndComp
-Wire Wire Line
-	5500 7700 5500 7650
-Connection ~ 5500 7650
+P 4950 7700
+F 0 "#PWR06" H 4950 7700 30  0001 C CNN
+F 1 "GND" H 4950 7630 30  0001 C CNN
+F 2 "" H 4950 7700 60  0000 C CNN
+F 3 "" H 4950 7700 60  0000 C CNN
+	1    4950 7700
+	1    0    0    -1
+$EndComp
 $Comp
 L GND #PWR07
@@
 Text GLabel 8050 1000 0    60   Input ~ 0
 Sensor+
-Text GLabel 8000 1850 0    60   Input ~ 0
-Sensor-
 Wire Wire Line
 	2800 1000 2750 1000
@@
 NoConn ~ 6350 7050
 NoConn ~ 6350 6950
-NoConn ~ 6000 7200
 $Comp
 L +3.3V #PWR016
@@
 	1    0    0    -1
 $EndComp
-Wire Wire Line
-	8000 1850 8200 1850
 $Comp
 L GND #PWR021
@@
 Wire Wire Line
 	8150 1850 8150 2100
-Connection ~ 8150 1850
 $Comp
 L R R21
@@
 P 7350 2550
 F 0 "Q3" H 7250 2700 60  0000 C CNN
-F 1 "MOSFET_N_P_CH" H 7850 2350 60  0000 C CNN
+F 1 "DMG6602SVT-7DICT-ND" H 8000 2350 60  0000 C CNN
 F 2 "kicad-libraries:SOT23-6" H 7250 2550 60  0001 C CNN
 F 3 "" H 7250 2550 60  0001 C CNN
@@
 P 7350 1300
 F 0 "Q3" H 7250 1450 60  0000 C CNN
-F 1 "MOSFET_N_P_CH" H 7200 1600 60  0001 C CNN
+F 1 "DMG6602SVT-7DICT-ND" H 7200 1600 60  0001 C CNN
 F 2 "kicad-libraries:SOT23-6" H 7250 1300 60  0001 C CNN
 F 3 "" H 7250 1300 60  0001 C CNN
@@
 	5000 5800 5100 5800
 Wire Wire Line
-	6200 2800 6200 2600
+	6200 2600 6200 2850
 Wire Wire Line
 	6200 2600 6150 2600
 Connection ~ 6200 2800
 Wire Wire Line
-	6200 1550 6200 1350
+	6200 1350 6200 1600
 Wire Wire Line
 	6200 1350 6150 1350
@@
 	2150 6450 1950 6450
 NoConn ~ 6350 6550
+$Comp
+L R R24
+U 1 1 5A99E358
+P 6200 3100
+F 0 "R24" H 6350 3200 50  0000 C CNN
+F 1 "10k" V 6200 3100 50  0000 C CNN
+F 2 "kicad-libraries:R0603F" H 6200 3100 60  0001 C CNN
+F 3 "" H 6200 3100 60  0000 C CNN
+	1    6200 3100
+	1    0    0    -1
+$EndComp
+$Comp
+L R R23
+U 1 1 5A99E63D
+P 6200 1850
+F 0 "R23" H 6350 1950 50  0000 C CNN
+F 1 "10k" V 6200 1850 50  0000 C CNN
+F 2 "kicad-libraries:R0603F" H 6200 1850 60  0001 C CNN
+F 3 "" H 6200 1850 60  0000 C CNN
+	1    6200 1850
+	1    0    0    -1
+$EndComp
+$Comp
+L GND #PWR022
+U 1 1 5A99F1FC
+P 6200 3400
+F 0 "#PWR022" H 6200 3400 30  0001 C CNN
+F 1 "GND" H 6200 3330 30  0001 C CNN
+F 2 "" H 6200 3400 60  0000 C CNN
+F 3 "" H 6200 3400 60  0000 C CNN
+	1    6200 3400
+	1    0    0    -1
+$EndComp
+$Comp
+L GND #PWR023
+U 1 1 5A99F2D6
+P 6200 2150
+F 0 "#PWR023" H 6200 2150 30  0001 C CNN
+F 1 "GND" H 6200 2080 30  0001 C CNN
+F 2 "" H 6200 2150 60  0000 C CNN
+F 3 "" H 6200 2150 60  0000 C CNN
+	1    6200 2150
+	1    0    0    -1
+$EndComp
+Wire Wire Line
+	6200 2100 6200 2150
+Wire Wire Line
+	6200 3350 6200 3400
+Wire Wire Line
+	8200 1850 8150 1850
+Wire Wire Line
+	1000 2850 4150 2850
+$Comp
+L GND #PWR024
+U 1 1 5A9A0922
+P 1500 2900
+F 0 "#PWR024" H 1500 2900 30  0001 C CNN
+F 1 "GND" H 1500 2830 30  0001 C CNN
+F 2 "" H 1500 2900 60  0000 C CNN
+F 3 "" H 1500 2900 60  0000 C CNN
+	1    1500 2900
+	1    0    0    -1
+$EndComp
 $EndSCHEMATC

Commit message: update documentation
Parts:
- P2: value MP-PWM-2 -> MP-GND
Changed lines of the file:
@@
 P 4800 5800
 F 0 "P2" H 4700 5850 50  0000 C CNN
-F 1 "MP-PWM-2" H 4850 5700 50  0000 C CNN
+F 1 "MP-GND" H 4850 5700 50  0000 C CNN
 F 2 "kicad-libraries:CONN_1" H 4800 5800 50  0001 C CNN
 F 3 "" H 4800 5800 50  0000 C CNN

Commit message: Korrektur pcb
Connections:
- net +UA: now also Q3.2 (S); no longer Q3.4 (D)
- net at LS1.1, P4.1 (P1), Q3.6 (D)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: now also Q3.4 (D); no longer Q3.2 (S)
Changed lines of the file:
@@
 	1    0    0    -1
 $EndComp
-Wire Wire Line
-	6550 1300 7150 1300
 Text GLabel 6100 1550 0    60   Input ~ 0
 PWM-1-OUT
@@
 Wire Wire Line
 	6550 700  6550 750
-Wire Wire Line
-	7450 700  7450 1100
-Wire Wire Line
-	7450 1500 7450 2350
 $Comp
 L MOSFET_N_P_CH Q3
@@
 U 2 1 5A98ECF2
 P 7350 1300
-F 0 "Q3" H 7250 1450 60  0000 C CNN
+F 0 "Q3" H 7200 1100 60  0000 C CNN
 F 1 "DMG6602SVT-7DICT-ND" H 7200 1600 60  0001 C CNN
 F 2 "kicad-libraries:SOT23-6" H 7250 1300 60  0001 C CNN
 F 3 "" H 7250 1300 60  0001 C CNN
 	2    7350 1300
-	1    0    0    -1
+	1    0    0    1
 $EndComp
 Wire Wire Line
@@
 	1    0    0    -1
 $EndComp
+Wire Wire Line
+	6550 1300 7150 1300
+Wire Wire Line
+	7450 700  7450 1100
+Wire Wire Line
+	7450 1500 7450 2350
 $EndSCHEMATC

Commit message: Schaltplan Korrektur
Parts:
- removed D1: ZENER, kicad-libraries:SOD-123, symbol ZENER
- removed Q2: MOSFET_N_CH, kicad-libraries:SOT23GDS, symbol MOSFET_N_CH
- removed R21: 1k, kicad-libraries:1206E, symbol R
Connections:
- net PWM-2-OUT: now also Q3.1 (G)
- net at P8.1 (P1), R30.2, U1.1 (OUT)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: now also RV1.3
- net at R6.1, RV1.2: now also RV1.1; no longer RV1.3
- net at R10.2: now also RV2.1; no longer RV2.2
- net at C6.2, R7.1, RV2.3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: now also RV2.2
Other:
- moved on the sheet: C10, C11, C14, C7, C8, P0, P2, P6, R24, RP1, RV1, RV2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
